File: EVO2513-0_5_0.kicad_sch (KiCad schematic)
At the start: 43 parts, among them J1 ${ALTIUM_VALUE}, J2 ${ALTIUM_VALUE}, J3 ${ALTIUM_VALUE}, J4 ${ALTIUM_VALUE}, J5 ${ALTIUM_VALUE}, J6 ${ALTIUM_VALUE}, M1 ${ALTIUM_VALUE}, M2 ${ALTIUM_VALUE}, M3 ${ALTIUM_VALUE}, M4 ${ALTIUM_VALUE}, M5 ${ALTIUM_VALUE}, M6 ${ALTIUM_VALUE}

Commit message: Replace ${ALTIUM_VALUE} placeholders with literal values
The Altium import left every symbol's Value field as ${ALTIUM_VALUE},
resolved through a per-symbol ALTIUM_VALUE field. Copy that field's
contents into Value (209 symbols) so values are visible in tools and
exports that don't resolve the variable. All values match the PCB.

The 26 BON pogo test pads had no ALTIUM_VALUE field; set them to POGO-1.

Co-Authored-By: Claude Opus 5.5 <noreply@anthropic.com>
Parts:
- BON1, BON10, BON11, BON12, BON13, BON14, BON15, BON16, BON17, BON18, BON19, BON2, BON20, BON21, BON22, BON23, BON24, BON25, BON26, BON3, BON4, BON5, BON6, BON7, BON8, BON9: value ${ALTIUM_VALUE} -> POGO-1
- J1: value ${ALTIUM_VALUE} -> 1053101204
- J2: value ${ALTIUM_VALUE} -> 1053101114
- J3: value ${ALTIUM_VALUE} -> 10144517-043802LF
- J4: value ${ALTIUM_VALUE} -> 1053102204
- J5, J6: value ${ALTIUM_VALUE} -> 1053091102
- M1, M2, M3, M4, M5, M6: value ${ALTIUM_VALUE} -> 78614150960
- R28: value ${ALTIUM_VALUE} -> 10K
- TH1, TH2: value ${ALTIUM_VALUE} -> 10k
Changed lines of the file:
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@@
 			)
 		)
-		(property "Value" "${ALTIUM_VALUE}"
+		(property "Value" "POGO-1"
 			(at 232.41 134.4422 0)
 			(hide yes)
@@
 			)
 		)
-		(property "Value" "${ALTIUM_VALUE}"
+		(property "Value" "POGO-1"
 			(at 232.41 130.6322 0)
 			(hide yes)
@@
 			)
 		)
-		(property "Value" "${ALTIUM_VALUE}"
+		(property "Value" "POGO-1"
 			(at 167.64 130.6322 0)
 			(hide yes)
@@
 			)
 		)
-		(property "Value" "${ALTIUM_VALUE}"
+		(property "Value" "10144517-043802LF"
 			(at 210.82 100.1522 0)
 			(hide yes)
@@
 			)
 		)
-		(property "Value" "${ALTIUM_VALUE}"
+		(property "Value" "1053101204"
 			(at 307.34 163.6522 0)
 			(hide yes)
@@
 			)
 		)
-		(property "Value" "${ALTIUM_VALUE}"
+		(property "Value" "1053091102"
 			(at 335.28 126.8222 0)
 			(hide yes)
@@
 			)
 		)
-		(property "Value" "${ALTIUM_VALUE}"
+		(property "Value" "POGO-1"
 			(at 167.64 161.1122 0)
 			(hide yes)
@@
 			)
 		)
-		(property "Value" "${ALTIUM_VALUE}"
+		(property "Value" "POGO-1"
 			(at 232.41 157.3022 0)
 			(hide yes)
@@
 			)
 		)
-		(property "Value" "${ALTIUM_VALUE}"
+		(property "Value" "POGO-1"
 			(at 232.41 161.1122 0)
 			(hide yes)
@@
 			)
 		)
-		(property "Value" "${ALTIUM_VALUE}"
+		(property "Value" "POGO-1"
 			(at 241.3 164.9222 0)
 			(hide yes)
@@
 			)
 		)
-		(property "Value" "${ALTIUM_VALUE}"
+		(property "Value" "78614150960"
 			(at 40.64 262.7122 0)
 			(hide yes)
@@
 			)
 		)
-		(property "Value" "${ALTIUM_VALUE}"
+		(property "Value" "POGO-1"
 			(at 30.48 237.3122 0)
 			(hide yes)
@@
 			)
 		)
-		(property "Value" "${ALTIUM_VALUE}"
+		(property "Value" "1053091102"
 			(at 335.28 95.0722 0)
 			(hide yes)
@@
 			)
 		)
-		(property "Value" "${ALTIUM_VALUE}"
+		(property "Value" "POGO-1"
 			(at 232.41 138.2522 0)
 			(hide yes)
@@
 			)
 		)
-		(property "Value" "${ALTIUM_VALUE}"
+		(property "Value" "POGO-1"
 			(at 167.64 138.2522 0)
 			(hide yes)
@@
 			)
 		)
-		(property "Value" "${ALTIUM_VALUE}"
+		(property "Value" "POGO-1"
 			(at 167.64 145.8722 0)
 			(hide yes)
@@
 			)
 		)
-		(property "Value" "${ALTIUM_VALUE}"
+		(property "Value" "POGO-1"
 			(at 167.64 157.3022 0)
 			(hide yes)
@@
 			)
 		)
-		(property "Value" "${ALTIUM_VALUE}"
+		(property "Value" "78614150960"
 			(at 83.82 262.7122 0)
 			(hide yes)
@@
 			)
 		)
-		(property "Value" "${ALTIUM_VALUE}"
+		(property "Value" "10K"
 			(at 230.124 168.2242 90)
 			(hide yes)
@@
 			)
 		)
-		(property "Value" "${ALTIUM_VALUE}"
+		(property "Value" "POGO-1"
 			(at 167.64 153.4922 0)
 			(hide yes)
@@
 			)
 		)
-		(property "Value" "${ALTIUM_VALUE}"
+		(property "Value" "POGO-1"
 			(at 232.41 123.0122 0)
 			(hide yes)
@@
 			)
 		)
-		(property "Value" "${ALTIUM_VALUE}"
+		(property "Value" "POGO-1"
 			(at 232.41 153.4922 0)
 			(hide yes)
@@
 			)
 		)
-		(property "Value" "${ALTIUM_VALUE}"
+		(property "Value" "POGO-1"
 			(at 232.41 100.1522 0)
 			(hide yes)
@@
 			)
 		)
-		(property "Value" "${ALTIUM_VALUE}"
+		(property "Value" "POGO-1"
 			(at 165.1 103.9622 0)
 			(hide yes)
@@
 			)
 		)
-		(property "Value" "${ALTIUM_VALUE}"
+		(property "Value" "78614150960"
 			(at 127 262.7122 0)
 			(hide yes)
@@
 			)
 		)
-		(property "Value" "${ALTIUM_VALUE}"
+		(property "Value" "POGO-1"
 			(at 167.64 126.8222 0)
 			(hide yes)
@@
 			)
 		)
-		(property "Value" "${ALTIUM_VALUE}"
+		(property "Value" "POGO-1"
 			(at 167.64 149.6822 0)
 			(hide yes)
@@
 			)
 		)
-		(property "Value" "${ALTIUM_VALUE}"
+		(property "Value" "10k"
 			(at 267.462 168.2242 90)
 			(hide yes)
@@
 			)
 		)
-		(property "Value" "${ALTIUM_VALUE}"
+		(property "Value" "POGO-1"
 			(at 167.64 164.9222 0)
 			(hide yes)
@@
 			)
 		)
-		(property "Value" "${ALTIUM_VALUE}"
+		(property "Value" "POGO-1"
 			(at 232.41 126.8222 0)
 			(hide yes)
@@
 			)
 		)
-		(property "Value" "${ALTIUM_VALUE}"
+		(property "Value" "1053101114"
 			(at 97.79 140.7922 0)
 			(hide yes)
@@
 			)
 		)
-		(property "Value" "${ALTIUM_VALUE}"
+		(property "Value" "1053102204"
 			(at 97.79 87.4522 0)
 			(hide yes)
@@
 			)
 		)
-		(property "Value" "${ALTIUM_VALUE}"
+		(property "Value" "10k"
 			(at 257.302 168.2242 90)
 			(hide yes)
@@
 			)
 		)
-		(property "Value" "${ALTIUM_VALUE}"
+		(property "Value" "POGO-1"
 			(at 232.41 115.3922 0)
 			(hide yes)
@@
 			)
 		)
-		(property "Value" "${ALTIUM_VALUE}"
+		(property "Value" "POGO-1"
 			(at 167.64 134.4422 0)
 			(hide yes)
@@
 			)
 		)
-		(property "Value" "${ALTIUM_VALUE}"
+		(property "Value" "78614150960"
 			(at 62.23 262.7122 0)
 			(hide yes)
@@
 			)
 		)
-		(property "Value" "${ALTIUM_VALUE}"
+		(property "Value" "78614150960"
 			(at 17.78 262.7122 0)
 			(hide yes)
@@
 			)
 		)
-		(property "Value" "${ALTIUM_VALUE}"
+		(property "Value" "POGO-1"
 			(at 232.41 149.6822 0)
 			(hide yes)
@@
 			)
 		)
-		(property "Value" "${ALTIUM_VALUE}"
+		(property "Value" "POGO-1"
 			(at 232.41 145.8722 0)
 			(hide yes)
@@
 			)
 		)
-		(property "Value" "${ALTIUM_VALUE}"
+		(property "Value" "78614150960"
 			(at 105.41 262.7122 0)
 			(hide yes)
@@
 			)
 		)
-		(property "Value" "${ALTIUM_VALUE}"
+		(property "Value" "POGO-1"
 			(at 17.78 237.3122 0)
 			(hide yes)

Commit message: Fix footprint name case mismatches between schematic and PCB
The Altium import wrote 12 symbol Footprint fields with different
letter case from the footprint actually placed on the PCB and stored
in the project library (e.g. "Ind Coilcraft XAL8080" vs
"IND COILCRAFT XAL8080"). Library lookup is case-sensitive, so these
footprints could not be found when updating the PCB from the schematic.

Point each field at the footprint the PCB uses: J2, J5, J6, M2-M6,
FL1, D9, D10 and L2. The PCB is unchanged.

Co-Authored-By: Claude Opus 5.5 <noreply@anthropic.com>
Parts:
- J2: footprint EVO2513-0_5_0-import-fps:Connector Molex 1053101114 2.5mm THP -> EVO2513-0_5_0-import-fps:CONNECTOR MOLEX 1053101114 2.5MM THP
- J5, J6: footprint EVO2513-0_5_0-import-fps:Connector Molex 1053091102 2POS 2.5mm THP -> EVO2513-0_5_0-import-fps:CONNECTOR MOLEX 1053091102 2POS 2.5MM THP
- M2, M3, M4, M5, M6: footprint EVO2513-0_5_0-import-fps:Mech Spacer Wurth 78614150960 Through M3 -> EVO2513-0_5_0-import-fps:MECH SPACER WURTH 78614150960 THROUGH M3
Changed lines of the file:
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@@
 			)
 		)
-		(property "Footprint" "EVO2513-0_5_0-import-fps:Connector Molex 1053091102 2POS 2.5mm THP"
+		(property "Footprint" "EVO2513-0_5_0-import-fps:CONNECTOR MOLEX 1053091102 2POS 2.5MM THP"
 			(at 322.58 124.2822 0)
 			(hide yes)
@@
 			)
 		)
-		(property "Footprint" "EVO2513-0_5_0-import-fps:Mech Spacer Wurth 78614150960 Through M3"
+		(property "Footprint" "EVO2513-0_5_0-import-fps:MECH SPACER WURTH 78614150960 THROUGH M3"
 			(at 40.64 267.7922 0)
 			(hide yes)
@@
 			)
 		)
-		(property "Footprint" "EVO2513-0_5_0-import-fps:Connector Molex 1053091102 2POS 2.5mm THP"
+		(property "Footprint" "EVO2513-0_5_0-import-fps:CONNECTOR MOLEX 1053091102 2POS 2.5MM THP"
 			(at 322.58 92.5322 0)
 			(hide yes)
@@
 			)
 		)
-		(property "Footprint" "EVO2513-0_5_0-import-fps:Mech Spacer Wurth 78614150960 Through M3"
+		(property "Footprint" "EVO2513-0_5_0-import-fps:MECH SPACER WURTH 78614150960 THROUGH M3"
 			(at 83.82 267.7922 0)
 			(hide yes)
@@
 			)
 		)
-		(property "Footprint" "EVO2513-0_5_0-import-fps:Mech Spacer Wurth 78614150960 Through M3"
+		(property "Footprint" "EVO2513-0_5_0-import-fps:MECH SPACER WURTH 78614150960 THROUGH M3"
 			(at 127 267.7922 0)
 			(hide yes)
@@
 			)
 		)
-		(property "Footprint" "EVO2513-0_5_0-import-fps:Connector Molex 1053101114 2.5mm THP"
+		(property "Footprint" "EVO2513-0_5_0-import-fps:CONNECTOR MOLEX 1053101114 2.5MM THP"
 			(at 85.09 138.2522 0)
 			(hide yes)
@@
 			)
 		)
-		(property "Footprint" "EVO2513-0_5_0-import-fps:Mech Spacer Wurth 78614150960 Through M3"
+		(property "Footprint" "EVO2513-0_5_0-import-fps:MECH SPACER WURTH 78614150960 THROUGH M3"
 			(at 62.23 267.7922 0)
 			(hide yes)
@@
 			)
 		)
-		(property "Footprint" "EVO2513-0_5_0-import-fps:Mech Spacer Wurth 78614150960 Through M3"
+		(property "Footprint" "EVO2513-0_5_0-import-fps:MECH SPACER WURTH 78614150960 THROUGH M3"
 			(at 105.41 267.7922 0)
 			(hide yes)

Commit message: Rename imported FOOTPRINT field to ALTIUM_FOOTPRINT
The Altium import added a user field named FOOTPRINT holding the bare
package name (e.g. "0402", "SMA"). KiCad matches field names
case-insensitively, so it overrode the real Footprint field: Update PCB
from Schematic looked up footprints like "0402" and failed for 222
parts, and saving the schematic replaced each library footprint link
with the package name.

Rename the field on all 237 symbols so the package name is kept but no
longer collides with Footprint.

Co-Authored-By: Claude Opus 5.5 <noreply@anthropic.com>
Parts:
- BON1, BON10, BON11, BON12, BON13, BON14, BON15, BON16, BON17, BON18, BON19, BON2, BON20, BON21, BON22, BON23, BON24, BON25, BON26, BON3, BON4, BON5, BON6, BON7, BON8, BON9: ALTIUM_FOOTPRINT (none) -> SMD 1.25mm; FOOTPRINT SMD 1.25mm -> (none)
- J1, J4, J5, J6: ALTIUM_FOOTPRINT (none) -> THP 2.5mm; FOOTPRINT THP 2.5mm -> (none)
- J2: ALTIUM_FOOTPRINT (none) -> 2.5mm THP Vert; FOOTPRINT 2.5mm THP Vert -> (none)
- J3: ALTIUM_FOOTPRINT (none) -> 0.8mm BergStak; FOOTPRINT 0.8mm BergStak -> (none)
- M1, M2, M3, M4, M5, M6: ALTIUM_FOOTPRINT (none) -> THP Through M3 15mm; FOOTPRINT THP Through M3 15mm -> (none)
- R28: ALTIUM_FOOTPRINT (none) -> 0402; FOOTPRINT 0402 -> (none)
- TH1, TH2: ALTIUM_FOOTPRINT (none) -> 0603; FOOTPRINT 0603 -> (none)
Changed lines of the file:
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@@
 			)
 		)
-		(property "FOOTPRINT" "SMD 1.25mm"
+		(property "ALTIUM_FOOTPRINT" "SMD 1.25mm"
 			(at 231.14 132.6642 0)
 			(hide yes)
@@
 			)
 		)
-		(property "FOOTPRINT" "SMD 1.25mm"
+		(property "ALTIUM_FOOTPRINT" "SMD 1.25mm"
 			(at 231.14 128.8542 0)
 			(hide yes)
@@
 			)
 		)
-		(property "FOOTPRINT" "SMD 1.25mm"
+		(property "ALTIUM_FOOTPRINT" "SMD 1.25mm"
 			(at 166.37 128.8542 0)
 			(hide yes)
@@
 			)
 		)
-		(property "FOOTPRINT" "0.8mm BergStak"
+		(property "ALTIUM_FOOTPRINT" "0.8mm BergStak"
 			(at 184.912 93.8022 0)
 			(hide yes)
@@
 			)
 		)
-		(property "FOOTPRINT" "THP 2.5mm"
+		(property "ALTIUM_FOOTPRINT" "THP 2.5mm"
 			(at 330.2 183.9722 0)
 			(hide yes)
@@
 			)
 		)
-		(property "FOOTPRINT" "THP 2.5mm"
+		(property "ALTIUM_FOOTPRINT" "THP 2.5mm"
 			(at 332.74 147.1422 0)
 			(hide yes)
@@
 			)
 		)
-		(property "FOOTPRINT" "SMD 1.25mm"
+		(property "ALTIUM_FOOTPRINT" "SMD 1.25mm"
 			(at 166.37 159.3342 0)
 			(hide yes)
@@
 			)
 		)
-		(property "FOOTPRINT" "SMD 1.25mm"
+		(property "ALTIUM_FOOTPRINT" "SMD 1.25mm"
 			(at 231.14 155.5242 0)
 			(hide yes)
@@
 			)
 		)
-		(property "FOOTPRINT" "SMD 1.25mm"
+		(property "ALTIUM_FOOTPRINT" "SMD 1.25mm"
 			(at 231.14 159.3342 0)
 			(hide yes)
@@
 			)
 		)
-		(property "FOOTPRINT" "SMD 1.25mm"
+		(property "ALTIUM_FOOTPRINT" "SMD 1.25mm"
 			(at 240.03 163.1442 0)
 			(hide yes)
@@
 			)
 		)
-		(property "FOOTPRINT" "THP Through M3 15mm"
+		(property "ALTIUM_FOOTPRINT" "THP Through M3 15mm"
 			(at 38.804 262.8392 0)
 			(hide yes)
@@
 			)
 		)
-		(property "FOOTPRINT" "SMD 1.25mm"
+		(property "ALTIUM_FOOTPRINT" "SMD 1.25mm"
 			(at 29.21 235.5342 0)
 			(hide yes)
@@
 			)
 		)
-		(property "FOOTPRINT" "THP 2.5mm"
+		(property "ALTIUM_FOOTPRINT" "THP 2.5mm"
 			(at 332.74 115.3922 0)
 			(hide yes)
@@
 			)
 		)
-		(property "FOOTPRINT" "SMD 1.25mm"
+		(property "ALTIUM_FOOTPRINT" "SMD 1.25mm"
 			(at 231.14 136.4742 0)
 			(hide yes)
@@
 			)
 		)
-		(property "FOOTPRINT" "SMD 1.25mm"
+		(property "ALTIUM_FOOTPRINT" "SMD 1.25mm"
 			(at 166.37 136.4742 0)
 			(hide yes)
@@
 			)
 		)
-		(property "FOOTPRINT" "SMD 1.25mm"
+		(property "ALTIUM_FOOTPRINT" "SMD 1.25mm"
 			(at 166.37 144.0942 0)
 			(hide yes)
@@
 			)
 		)
-		(property "FOOTPRINT" "SMD 1.25mm"
+		(property "ALTIUM_FOOTPRINT" "SMD 1.25mm"
 			(at 166.37 155.5242 0)
 			(hide yes)
@@
 			)
 		)
-		(property "FOOTPRINT" "THP Through M3 15mm"
+		(property "ALTIUM_FOOTPRINT" "THP Through M3 15mm"
 			(at 81.984 262.8392 0)
 			(hide yes)
@@
 			)
 		)
-		(property "FOOTPRINT" "0402"
+		(property "ALTIUM_FOOTPRINT" "0402"
 			(at 232.156 177.1142 90)
 			(show_name no)
@@
 			)
 		)
-		(property "FOOTPRINT" "SMD 1.25mm"
+		(property "ALTIUM_FOOTPRINT" "SMD 1.25mm"
 			(at 166.37 151.7142 0)
 			(hide yes)
@@
 			)
 		)
-		(property "FOOTPRINT" "SMD 1.25mm"
+		(property "ALTIUM_FOOTPRINT" "SMD 1.25mm"
 			(at 231.14 121.2342 0)
 			(hide yes)
@@
 			)
 		)
-		(property "FOOTPRINT" "SMD 1.25mm"
+		(property "ALTIUM_FOOTPRINT" "SMD 1.25mm"
 			(at 231.14 151.7142 0)
 			(hide yes)
@@
 			)
 		)
-		(property "FOOTPRINT" "SMD 1.25mm"
+		(property "ALTIUM_FOOTPRINT" "SMD 1.25mm"
 			(at 231.14 98.3742 0)
 			(hide yes)
@@
 			)
 		)
-		(property "FOOTPRINT" "SMD 1.25mm"
+		(property "ALTIUM_FOOTPRINT" "SMD 1.25mm"
 			(at 163.83 102.1842 0)
 			(hide yes)
@@
 			)
 		)
-		(property "FOOTPRINT" "THP Through M3 15mm"
+		(property "ALTIUM_FOOTPRINT" "THP Through M3 15mm"
 			(at 125.164 262.8392 0)
 			(hide yes)
@@
 			)
 		)
-		(property "FOOTPRINT" "SMD 1.25mm"
+		(property "ALTIUM_FOOTPRINT" "SMD 1.25mm"
 			(at 166.37 125.0442 0)
 			(hide yes)
@@
 			)
 		)
-		(property "FOOTPRINT" "SMD 1.25mm"
+		(property "ALTIUM_FOOTPRINT" "SMD 1.25mm"
 			(at 166.37 147.9042 0)
 			(hide yes)
@@
 			)
 		)
-		(property "FOOTPRINT" "0603"
+		(property "ALTIUM_FOOTPRINT" "0603"
 			(at 271.018 177.1142 90)
 			(show_name no)
@@
 			)
 		)
-		(property "FOOTPRINT" "SMD 1.25mm"
+		(property "ALTIUM_FOOTPRINT" "SMD 1.25mm"
 			(at 166.37 163.1442 0)
 			(hide yes)
@@
 			)
 		)
-		(property "FOOTPRINT" "SMD 1.25mm"
+		(property "ALTIUM_FOOTPRINT" "SMD 1.25mm"
 			(at 231.14 125.0442 0)
 			(hide yes)
@@
 			)
 		)
-		(property "FOOTPRINT" "2.5mm THP Vert"
+		(property "ALTIUM_FOOTPRINT" "2.5mm THP Vert"
 			(at 95.25 161.1122 0)
 			(hide yes)
@@
 			)
 		)
-		(property "FOOTPRINT" "THP 2.5mm"
+		(property "ALTIUM_FOOTPRINT" "THP 2.5mm"
 			(at 95.25 107.7722 0)
 			(hide yes)
@@
 			)
 		)
-		(property "FOOTPRINT" "0603"
+		(property "ALTIUM_FOOTPRINT" "0603"
 			(at 260.858 177.1142 90)
 			(show_name no)
@@
 			)
 		)
-		(property "FOOTPRINT" "SMD 1.25mm"
+		(property "ALTIUM_FOOTPRINT" "SMD 1.25mm"
 			(at 231.14 113.6142 0)
 			(hide yes)
@@
 			)
 		)
-		(property "FOOTPRINT" ""
+		(property "ALTIUM_FOOTPRINT" ""
 			(at 15.24 291.9222 0)
 			(hide yes)
@@
 			)
 		)
-		(property "FOOTPRINT" "SMD 1.25mm"
+		(property "ALTIUM_FOOTPRINT" "SMD 1.25mm"
 			(at 166.37 132.6642 0)
 			(hide yes)
@@
 			)
 		)
-		(property "FOOTPRINT" "THP Through M3 15mm"
+		(property "ALTIUM_FOOTPRINT" "THP Through M3 15mm"
 			(at 60.394 262.8392 0)
 			(hide yes)
@@
 			)
 		)
-		(property "FOOTPRINT" ""
+		(property "ALTIUM_FOOTPRINT" ""
 			(at 15.24 289.3822 0)
 			(hide yes)
@@
 			)
 		)
-		(property "FOOTPRINT" "THP Through M3 15mm"
+		(property "ALTIUM_FOOTPRINT" "THP Through M3 15mm"
 			(at 15.944 270.3322 0)
 			(hide yes)
@@
 			)
 		)
-		(property "FOOTPRINT" "SMD 1.25mm"
+		(property "ALTIUM_FOOTPRINT" "SMD 1.25mm"
 			(at 231.14 147.9042 0)
 			(hide yes)
@@
 			)
 		)
-		(property "FOOTPRINT" "SMD 1.25mm"
+		(property "ALTIUM_FOOTPRINT" "SMD 1.25mm"
 			(at 231.14 144.0942 0)
 			(hide yes)
@@
 			)
 		)
-		(property "FOOTPRINT" "THP Through M3 15mm"
+		(property "ALTIUM_FOOTPRINT" "THP Through M3 15mm"
 			(at 103.574 262.8392 0)
 			(hide yes)
@@
 			)
 		)
-		(property "FOOTPRINT" "SMD 1.25mm"
+		(property "ALTIUM_FOOTPRINT" "SMD 1.25mm"
 			(at 16.51 235.5342 0)
 			(hide yes)
