File: S02 Input Protection.kicad_sch (KiCad schematic)
At the start: 14 parts, among them Q1 ${ALTIUM_VALUE}, Q3 ${ALTIUM_VALUE}, U2 ${ALTIUM_VALUE}

Commit message: Replace ${ALTIUM_VALUE} placeholders with literal values
The Altium import left every symbol's Value field as ${ALTIUM_VALUE},
resolved through a per-symbol ALTIUM_VALUE field. Copy that field's
contents into Value (209 symbols) so values are visible in tools and
exports that don't resolve the variable. All values match the PCB.

The 26 BON pogo test pads had no ALTIUM_VALUE field; set them to POGO-1.

Co-Authored-By: Claude Opus 5.5 <noreply@anthropic.com>
Parts:
- C1: value ${ALTIUM_VALUE} -> 4.7nF
- D1: value ${ALTIUM_VALUE} -> 1.5SMB27CA
- FL1: value ${ALTIUM_VALUE} -> BNX024H01L
- LED1: value ${ALTIUM_VALUE} -> QTLP600C-4
- Q1, Q3: value ${ALTIUM_VALUE} -> DMT4011LFG
- R1: value ${ALTIUM_VALUE} -> 620K
- R2: value ${ALTIUM_VALUE} -> 12K
- R3: value ${ALTIUM_VALUE} -> 100K
- R4, R5: value ${ALTIUM_VALUE} -> 10R
- R6: value ${ALTIUM_VALUE} -> 5.1K
- R7: value ${ALTIUM_VALUE} -> 10K
- U2: value ${ALTIUM_VALUE} -> LTC4365
Changed lines of the file:
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@@
 			)
 		)
-		(property "Value" "${ALTIUM_VALUE}"
+		(property "Value" "BNX024H01L"
 			(at 271.78 97.6122 0)
 			(hide yes)
@@
 			)
 		)
-		(property "Value" "${ALTIUM_VALUE}"
+		(property "Value" "620K"
 			(at 124.714 147.9042 90)
 			(hide yes)
@@
 			)
 		)
-		(property "Value" "${ALTIUM_VALUE}"
+		(property "Value" "4.7nF"
 			(at 199.39 177.6222 90)
 			(hide yes)
@@
 			)
 		)
-		(property "Value" "${ALTIUM_VALUE}"
+		(property "Value" "12K"
 			(at 124.714 165.6842 90)
 			(hide yes)
@@
 			)
 		)
-		(property "Value" "${ALTIUM_VALUE}"
+		(property "Value" "10R"
 			(at 200.914 125.0442 90)
 			(hide yes)
@@
 			)
 		)
-		(property "Value" "${ALTIUM_VALUE}"
+		(property "Value" "LTC4365"
 			(at 186.69 149.6822 0)
 			(hide yes)
@@
 			)
 		)
-		(property "Value" "${ALTIUM_VALUE}"
+		(property "Value" "QTLP600C-4"
 			(at 295.91 119.9642 90)
 			(hide yes)
@@
 			)
 		)
-		(property "Value" "${ALTIUM_VALUE}"
+		(property "Value" "1.5SMB27CA"
 			(at 107.95 130.1242 90)
 			(hide yes)
@@
 			)
 		)
-		(property "Value" "${ALTIUM_VALUE}"
+		(property "Value" "DMT4011LFG"
 			(at 219.71 98.8822 0)
 			(hide yes)
@@
 			)
 		)
-		(property "Value" "${ALTIUM_VALUE}"
+		(property "Value" "10K"
 			(at 296.164 107.2642 90)
 			(hide yes)
@@
 			)
 		)
-		(property "Value" "${ALTIUM_VALUE}"
+		(property "Value" "5.1K"
 			(at 200.914 159.3342 90)
 			(hide yes)
@@
 			)
 		)
-		(property "Value" "${ALTIUM_VALUE}"
+		(property "Value" "100K"
 			(at 139.954 140.2842 90)
 			(hide yes)
@@
 			)
 		)
-		(property "Value" "${ALTIUM_VALUE}"
+		(property "Value" "DMT4011LFG"
 			(at 167.64 98.8822 0)
 			(hide yes)
@@
 			)
 		)
-		(property "Value" "${ALTIUM_VALUE}"
+		(property "Value" "10R"
 			(at 184.404 125.0442 90)
 			(hide yes)

Commit message: Fix footprint name case mismatches between schematic and PCB
The Altium import wrote 12 symbol Footprint fields with different
letter case from the footprint actually placed on the PCB and stored
in the project library (e.g. "Ind Coilcraft XAL8080" vs
"IND COILCRAFT XAL8080"). Library lookup is case-sensitive, so these
footprints could not be found when updating the PCB from the schematic.

Point each field at the footprint the PCB uses: J2, J5, J6, M2-M6,
FL1, D9, D10 and L2. The PCB is unchanged.

Co-Authored-By: Claude Opus 5.5 <noreply@anthropic.com>
Parts:
- FL1: footprint EVO2513-0_5_0-import-fps:FILTER BNX0xxH01 -> EVO2513-0_5_0-import-fps:FILTER BNX0XXH01
Changed lines of the file:
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@@
 			)
 		)
-		(property "Footprint" "EVO2513-0_5_0-import-fps:FILTER BNX0xxH01"
+		(property "Footprint" "EVO2513-0_5_0-import-fps:FILTER BNX0XXH01"
 			(at 259.08 100.1522 0)
 			(hide yes)

Commit message: Rename imported FOOTPRINT field to ALTIUM_FOOTPRINT
The Altium import added a user field named FOOTPRINT holding the bare
package name (e.g. "0402", "SMA"). KiCad matches field names
case-insensitively, so it overrode the real Footprint field: Update PCB
from Schematic looked up footprints like "0402" and failed for 222
parts, and saving the schematic replaced each library footprint link
with the package name.

Rename the field on all 237 symbols so the package name is kept but no
longer collides with Footprint.

Co-Authored-By: Claude Opus 5.5 <noreply@anthropic.com>
Parts:
- C1, R1, R2, R3, R4, R5, R6, R7: ALTIUM_FOOTPRINT (none) -> 0402; FOOTPRINT 0402 -> (none)
- D1: ALTIUM_FOOTPRINT (none) -> DO-214AA; FOOTPRINT DO-214AA -> (none)
- FL1: ALTIUM_FOOTPRINT (none) -> BNX0xxH01; FOOTPRINT BNX0xxH01 -> (none)
- LED1: ALTIUM_FOOTPRINT (none) -> 0603; FOOTPRINT 0603 -> (none)
- Q1, Q3: ALTIUM_FOOTPRINT (none) -> Power DI3333-8; FOOTPRINT Power DI3333-8 -> (none)
- U2: ALTIUM_FOOTPRINT (none) -> 8-Pin DFN; FOOTPRINT 8-Pin DFN -> (none)
Changed lines of the file:
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@@
 			)
 		)
-		(property "FOOTPRINT" "BNX0xxH01"
+		(property "ALTIUM_FOOTPRINT" "BNX0xxH01"
 			(at 267.97 91.2622 0)
 			(hide yes)
@@
 			)
 		)
-		(property "FOOTPRINT" "0402"
+		(property "ALTIUM_FOOTPRINT" "0402"
 			(at 126.746 156.7942 90)
 			(show_name no)
@@
 			)
 		)
-		(property "FOOTPRINT" "0402"
+		(property "ALTIUM_FOOTPRINT" "0402"
 			(at 203.2 179.4002 90)
 			(show_name no)
@@
 			)
 		)
-		(property "FOOTPRINT" "0402"
+		(property "ALTIUM_FOOTPRINT" "0402"
 			(at 126.746 174.5742 90)
 			(show_name no)
@@
 			)
 		)
-		(property "FOOTPRINT" "0402"
+		(property "ALTIUM_FOOTPRINT" "0402"
 			(at 202.946 133.9342 90)
 			(show_name no)
@@
 			)
 		)
-		(property "FOOTPRINT" "8-Pin DFN"
+		(property "ALTIUM_FOOTPRINT" "8-Pin DFN"
 			(at 163.83 150.6982 0)
 			(hide yes)
@@
 			)
 		)
-		(property "FOOTPRINT" "0603"
+		(property "ALTIUM_FOOTPRINT" "0603"
 			(at 299.72 131.1402 90)
 			(show_name no)
@@
 			)
 		)
-		(property "FOOTPRINT" "DO-214AA"
+		(property "ALTIUM_FOOTPRINT" "DO-214AA"
 			(at 110.49 138.7602 90)
 			(show_name no)
@@
 			)
 		)
-		(property "FOOTPRINT" "Power DI3333-8"
+		(property "ALTIUM_FOOTPRINT" "Power DI3333-8"
 			(at 196.85 99.8982 0)
 			(hide yes)
@@
 			)
 		)
-		(property "FOOTPRINT" "0402"
+		(property "ALTIUM_FOOTPRINT" "0402"
 			(at 298.196 116.1542 90)
 			(show_name no)
@@
 			)
 		)
-		(property "FOOTPRINT" "0402"
+		(property "ALTIUM_FOOTPRINT" "0402"
 			(at 202.946 168.2242 90)
 			(show_name no)
@@
 			)
 		)
-		(property "FOOTPRINT" "0402"
+		(property "ALTIUM_FOOTPRINT" "0402"
 			(at 141.986 149.1742 90)
 			(show_name no)
@@
 			)
 		)
-		(property "FOOTPRINT" "Power DI3333-8"
+		(property "ALTIUM_FOOTPRINT" "Power DI3333-8"
 			(at 190.5 99.8982 0)
 			(hide yes)
@@
 			)
 		)
-		(property "FOOTPRINT" "0402"
+		(property "ALTIUM_FOOTPRINT" "0402"
 			(at 186.436 133.9342 90)
 			(show_name no)
