File: S02 Input Protection.kicad_sch (KiCad schematic)
At the start: 14 parts, among them Q1 DMT4011LFG, Q3 DMT4011LFG, U2 LTC4365

Commit message: Use KiCad standard footprints for chip resistors and capacitors
The imported Lattech R/C footprints have poor land patterns (the 0402s
use 0.635 mm circular pads) and cause tombstoning in assembly. Replace
all 139 chip resistors and capacitors with KiCad's standard IPC-7351
nominal footprints:

  Res 0402/0603/1206/2512 -> Resistor_SMD:R_xxxx_xxxxMetric (87)
  Cap 0402/0603/0805/1206/1210 -> Capacitor_SMD:C_xxxx_xxxxMetric (52)

Each part keeps its position, rotation, side, pad nets, schematic link
and reference/value text placement. The pads are on the same axis with
pad 1 on the same side, and every old pad centre lies inside the new
pad, so existing tracks still connect. Zones are refilled.

Schematic Footprint fields and the symbols' footprint filters point at
the new footprints, and the unused imported R/C footprints are removed
from the project library. Electrolytic capacitors are not changed.

DRC: 0 unconnected items, as before. Tracks, vias, zone outlines and
all other footprints are unchanged. 11 courtyard overlaps are new,
because the old footprints had no courtyards.

Co-Authored-By: Claude Opus 5.5 <noreply@anthropic.com>
Parts:
- C1: footprint EVO2513-0_5_0-import-fps:Cap 0402 H0-6 R -> Capacitor_SMD:C_0402_1005Metric
- R1, R2, R3, R4, R5, R6, R7: footprint EVO2513-0_5_0-import-fps:Res 0402 H0-45 R -> Resistor_SMD:R_0402_1005Metric
Changed lines of the file:
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@@
 			)
 		)
-		(property "Footprint" "EVO2513-0_5_0-import-fps:Res 0402 H0-45 R"
+		(property "Footprint" "Resistor_SMD:R_0402_1005Metric"
 			(at 125.73 152.2222 0)
 			(hide yes)
@@
 			)
 		)
-		(property "Footprint" "EVO2513-0_5_0-import-fps:Cap 0402 H0-6 R"
+		(property "Footprint" "Capacitor_SMD:C_0402_1005Metric"
 			(at 201.93 175.0822 0)
 			(hide yes)
@@
 			)
 		)
-		(property "Footprint" "EVO2513-0_5_0-import-fps:Res 0402 H0-45 R"
+		(property "Footprint" "Resistor_SMD:R_0402_1005Metric"
 			(at 125.73 170.0022 0)
 			(hide yes)
@@
 			)
 		)
-		(property "Footprint" "EVO2513-0_5_0-import-fps:Res 0402 H0-45 R"
+		(property "Footprint" "Resistor_SMD:R_0402_1005Metric"
 			(at 201.93 129.3622 0)
 			(hide yes)
@@
 			)
 		)
-		(property "Footprint" "EVO2513-0_5_0-import-fps:Res 0402 H0-45 R"
+		(property "Footprint" "Resistor_SMD:R_0402_1005Metric"
 			(at 297.18 111.5822 0)
 			(hide yes)
@@
 			)
 		)
-		(property "Footprint" "EVO2513-0_5_0-import-fps:Res 0402 H0-45 R"
+		(property "Footprint" "Resistor_SMD:R_0402_1005Metric"
 			(at 201.93 163.6522 0)
 			(hide yes)
@@
 			)
 		)
-		(property "Footprint" "EVO2513-0_5_0-import-fps:Res 0402 H0-45 R"
+		(property "Footprint" "Resistor_SMD:R_0402_1005Metric"
 			(at 140.97 144.6022 0)
 			(hide yes)
@@
 			)
 		)
-		(property "Footprint" "EVO2513-0_5_0-import-fps:Res 0402 H0-45 R"
+		(property "Footprint" "Resistor_SMD:R_0402_1005Metric"
 			(at 185.42 129.3622 0)
 			(hide yes)

Commit message: Fix schematic ERC issues from the import
ERC across all seven sheets reported 1481 issues from the import:

- Every item sat 43 mil off KiCad's 50 mil connection grid in Y, so new
  wires would not snap to existing pins. Each sheet's contents are
  shifted 7 mil (0.1778 mm) onto the grid; the library symbol
  definitions are untouched and a uniform shift keeps every connection.
  A few wire corners on S06 were off grid on their own (at 6740 mil,
  7620 mil and y 3290 mil); they move to the nearest grid point, which
  removes two 10 mil stubs and moves #PWR065 with its wire.
- Nine wires ran 1.27-2.54 mm past the label sitting on them (ID on S01;
  LDVR1/2 and HDVR1/2 on S06), leaving dangling ends. They are trimmed
  back to the label.
- GND, +12V, +3V3MCU and +5V enter through connector pins, so ERC had
  no power source for them. A PWR_FLAG (#FLG01-#FLG04) sits on each.
- The title-block module name used the Altium formula
  ${COPY(DOCUMENTNAME,5,LENGTH(DOCUMENTNAME)-11)}, which KiCad cannot
  evaluate. Each sheet now carries the title it produced.

ERC: 1481 -> 0. The netlist still matches the PCB's 147 nets.

Update PCB from Schematic was rerun afterwards. It changes metadata only:
footprint filters, unit and pin-function data from the symbols, and the
KiLib_Generator fields dropped from the 139 standard R/C footprints. No
placement or copper changes.

Co-Authored-By: Claude Opus 5.5 <noreply@anthropic.com>
Other:
- note added: "Input Protection"
- note removed: "${COPY(DOCUMENTNAME,5,LENGTH(DOCUMENTNAME)-11)}"

Commit message: Convert the schematic to a hierarchical root sheet
The Altium import produced seven KiCad 10 top-level sheets, with S01's
content in EVO2513-0_5_0.kicad_sch. kicad-cli only loads the first of
those, so command-line ERC, netlist and DRC parity checks saw S01 alone.

- EVO2513-0_5_0.kicad_sch is now a root sheet holding one sheet symbol per
  sheet; S01's content moves to "S01 External Connectors.kicad_sch".
- Each sheet symbol keeps its old top-level sheet UUID, so symbol
  references, net names and connectivity are unchanged: the netlist from
  the new root is identical to the previous whole-design netlist (229
  components, 147 nets). Cross-sheet nets still use global labels.
- The board's 229 footprint paths take the hierarchical form
  /<sheet>/<symbol>, and S01's footprints point at the new sheet file.
  No copper or placement changes.
- Every title block read "sheet 7 of 7" (a single DOCUMENTNUMBER project
  variable). Sheet numbers now use the page number: the root is page 1
  and S01-S07 are pages 2-8.

kicad-cli ERC over the whole design: 0 errors, 0 warnings. DRC with
schematic parity: 0 parity issues, 450 violations as before.

Co-Authored-By: Claude Opus 5.5 <noreply@anthropic.com>
Other:
- note added: "${#}"
- note removed: "${DOCUMENTNUMBER}"
Changed lines of the file:
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@@
 		)
 	)
-	(text "${DOCUMENTNUMBER}"
+	(text "${#}"
 		(exclude_from_sim no)
 		(at 298.45 292.1 0)
@@
 		(instances
 			(project "EVO2513-0_5_0"
-				(path "/8d5ba2ad-b155-424d-98b9-d2b0a3724e07"
+				(path "/44203427-0a3b-455b-9bb9-c1b577d179b3/8d5ba2ad-b155-424d-98b9-d2b0a3724e07"
 					(reference "FL1")
 					(unit 1)
@@
 		(instances
 			(project "EVO2513-0_5_0"
-				(path "/8d5ba2ad-b155-424d-98b9-d2b0a3724e07"
+				(path "/44203427-0a3b-455b-9bb9-c1b577d179b3/8d5ba2ad-b155-424d-98b9-d2b0a3724e07"
 					(reference "R1")
 					(unit 1)
@@
 		(instances
 			(project "EVO2513-0_5_0"
-				(path "/8d5ba2ad-b155-424d-98b9-d2b0a3724e07"
+				(path "/44203427-0a3b-455b-9bb9-c1b577d179b3/8d5ba2ad-b155-424d-98b9-d2b0a3724e07"
 					(reference "C1")
 					(unit 1)
@@
 		(instances
 			(project "EVO2513-0_5_0"
-				(path "/8d5ba2ad-b155-424d-98b9-d2b0a3724e07"
+				(path "/44203427-0a3b-455b-9bb9-c1b577d179b3/8d5ba2ad-b155-424d-98b9-d2b0a3724e07"
 					(reference "R2")
 					(unit 1)
@@
 		(instances
 			(project "EVO2513-0_5_0"
-				(path "/8d5ba2ad-b155-424d-98b9-d2b0a3724e07"
+				(path "/44203427-0a3b-455b-9bb9-c1b577d179b3/8d5ba2ad-b155-424d-98b9-d2b0a3724e07"
 					(reference "R5")
 					(unit 1)
@@
 		(instances
 			(project "EVO2513-0_5_0"
-				(path "/8d5ba2ad-b155-424d-98b9-d2b0a3724e07"
+				(path "/44203427-0a3b-455b-9bb9-c1b577d179b3/8d5ba2ad-b155-424d-98b9-d2b0a3724e07"
 					(reference "U2")
 					(unit 1)
@@
 		(instances
 			(project "EVO2513-0_5_0"
-				(path "/8d5ba2ad-b155-424d-98b9-d2b0a3724e07"
+				(path "/44203427-0a3b-455b-9bb9-c1b577d179b3/8d5ba2ad-b155-424d-98b9-d2b0a3724e07"
 					(reference "LED1")
 					(unit 1)
@@
 		(instances
 			(project "EVO2513-0_5_0"
-				(path "/8d5ba2ad-b155-424d-98b9-d2b0a3724e07"
+				(path "/44203427-0a3b-455b-9bb9-c1b577d179b3/8d5ba2ad-b155-424d-98b9-d2b0a3724e07"
 					(reference "D1")
 					(unit 1)
@@
 		(instances
 			(project "EVO2513-0_5_0"
-				(path "/8d5ba2ad-b155-424d-98b9-d2b0a3724e07"
+				(path "/44203427-0a3b-455b-9bb9-c1b577d179b3/8d5ba2ad-b155-424d-98b9-d2b0a3724e07"
 					(reference "Q3")
 					(unit 1)
@@
 		(instances
 			(project "EVO2513-0_5_0"
-				(path "/8d5ba2ad-b155-424d-98b9-d2b0a3724e07"
+				(path "/44203427-0a3b-455b-9bb9-c1b577d179b3/8d5ba2ad-b155-424d-98b9-d2b0a3724e07"
 					(reference "R7")
 					(unit 1)
@@
 		(instances
 			(project "EVO2513-0_5_0"
-				(path "/8d5ba2ad-b155-424d-98b9-d2b0a3724e07"
+				(path "/44203427-0a3b-455b-9bb9-c1b577d179b3/8d5ba2ad-b155-424d-98b9-d2b0a3724e07"
 					(reference "#PWR020")
 					(unit 1)
@@
 		(instances
 			(project "EVO2513-0_5_0"
-				(path "/8d5ba2ad-b155-424d-98b9-d2b0a3724e07"
+				(path "/44203427-0a3b-455b-9bb9-c1b577d179b3/8d5ba2ad-b155-424d-98b9-d2b0a3724e07"
 					(reference "R6")
 					(unit 1)
@@
 		(instances
 			(project "EVO2513-0_5_0"
-				(path "/8d5ba2ad-b155-424d-98b9-d2b0a3724e07"
+				(path "/44203427-0a3b-455b-9bb9-c1b577d179b3/8d5ba2ad-b155-424d-98b9-d2b0a3724e07"
 					(reference "R3")
 					(unit 1)
@@
 		(instances
 			(project "EVO2513-0_5_0"
-				(path "/8d5ba2ad-b155-424d-98b9-d2b0a3724e07"
+				(path "/44203427-0a3b-455b-9bb9-c1b577d179b3/8d5ba2ad-b155-424d-98b9-d2b0a3724e07"
 					(reference "Q1")
 					(unit 1)
@@
 		(instances
 			(project "EVO2513-0_5_0"
-				(path "/8d5ba2ad-b155-424d-98b9-d2b0a3724e07"
+				(path "/44203427-0a3b-455b-9bb9-c1b577d179b3/8d5ba2ad-b155-424d-98b9-d2b0a3724e07"
 					(reference "R4")
 					(unit 1)
@@
 		)
 	)
-	(sheet_instances
-		(path "/"
-			(page "2")
-		)
-	)

Commit message: Link the sheets through hierarchical labels and sheet pins
The 78 cross-sheet global labels on S01-S07 become hierarchical labels,
and each sheet symbol on the root gets a pin per label name (71 pins).
On the root, each pin connects through a short wire to a global label
with the net name. Global labels there, rather than local ones, keep the
35 net names free of a "/" sheet-path prefix, so the net classes and the
board's nets are unchanged.

Layout: S01 External Connectors on the left with its pins on the right
edge; S02-S04 and S05-S07 in two columns with their pins on the left.

The netlist is identical to before (229 components, 147 nets, same names
and pins). kicad-cli ERC: 0 errors, 0 warnings. DRC with schematic
parity: 0 parity issues, 450 violations as before.

Co-Authored-By: Claude Opus 5.5 <noreply@anthropic.com>
Changed lines of the file:
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@@
 		)
 	)
-	(global_label "GDINPUT"
+	(hierarchical_label "GDINPUT"
 		(shape passive)
 		(at 69.85 110.49 180)
-		(fields_autoplaced yes)
 		(effects
 			(font
@@
 			(justify right)
 		)
-		(property "Intersheetrefs" "${INTERSHEET_REFS}"
-			(at 69.85 110.49 0)
-			(effects
-				(font
-					(size 1.27 1.27)
-				)
-				(justify right)
-				(hide yes)
-			)
-		)
 	)
-	(global_label "DCFILTERED"
+	(hierarchical_label "DCFILTERED"
 		(shape passive)
 		(at 320.04 100.33 0)
-		(fields_autoplaced yes)
 		(effects
 			(font
@@
 			(justify left)
 		)
-		(property "Intersheetrefs" "${INTERSHEET_REFS}"
-			(at 320.04 100.33 0)
-			(effects
-				(font
-					(size 1.27 1.27)
-				)
-				(justify left)
-				(hide yes)
-			)
-		)
 	)
-	(global_label "DCINPUT"
+	(hierarchical_label "DCINPUT"
 		(shape passive)
 		(at 69.85 100.33 180)
-		(fields_autoplaced yes)
 		(effects
 			(font
@@
 			(justify right)
 		)
-		(property "Intersheetrefs" "${INTERSHEET_REFS}"
-			(at 69.85 100.33 0)
-			(effects
-				(font
-					(size 1.27 1.27)
-				)
-				(justify right)
-				(hide yes)
-			)
-		)
 	)
