File: S02 Input Protection.kicad_sch (KiCad schematic)
At the start: 14 parts, among them Q1 DMT6007LFGQ-7, Q3 DMT6007LFGQ-7, U2 LTC4365

Commit message: Raise divider impedances, dim the PG LEDs, use standard diode lands
TI asks for a pull-up of at least 350 kOhm on EN/UVLO above 5 V.
R108 100K -> 619K and R49 12K -> 75K, both values already on the
BOM: turn-on 11.10 V (10.63-11.91 V worst case), off 10.09 V. 1M/120K
was rejected because leakage across 1M puts worst-case turn-on at
12.24 V, above the rail.

Q24 gate bias R109 100K -> 1.07M and R110 27K -> 390K: +12V draw
94 -> 8.2 uA, gate 3.2 V at 12 V and under 4 V worst case at the
14.7 V OVLO limit. The R115 bypass pull-down is now 62.9K.

PGTH dividers R59/R61/R76 100K -> 390K and R60/R62/R77 13K -> 51K:
PG at 10.38 V (11.17 V worst case), 23.5 uA at threshold to meet TI's
20x PGTH leakage rule. 390K is the only new BOM value.

PG LED resistors R67/R68/R81 2.2K -> 4.7K, about 0.9 mA less on
battery with all rails up.

D1, D4, D6-D10 and LED1-LED4 move from imported Altium lands to KiCad
standard footprints (D_SMB, D_SMA, SOT-23, Diodes_UDFN-10, LED_0603),
in place with the same nets; the LEDs turn 180 deg for pad 1. Drops
the 8 thin LED A/C silk warnings. Five unused imported footprints
removed. Nearby parts and tracks adjusted for the new lands.

Keep the GND planes free of power copper, as on the original: remove
the SW1/L2 and SW2 strip zones and the small +12V (via block by R115)
and U5 ISNSP (under Q18's drain) zones from In1/In3/In5/In6. They
carried no current; GND gains about 0.8 mm2 on In1, 3.5 mm2 on In3
and In5 and 3.7 mm2 on In6 under the power stage.

Remove the 347 via-block octagons the Altium import left as copper
graphic polygons (gr_poly) on B.Cu and In1-In6, one 1.2 x 1.8 mm
octagon per six-via block per layer. As drawings they bypassed zone
rules, and on the GND layers they were net islands in the pour,
including the charger switch node. None carried current: same-net
pours connect the vias solid, and DRC finds 0 unconnected. GND gains
about 26 mm2 on In1, 21 mm2 on In3 and In5, 18 mm2 on In6 and 27 mm2
on B.Cu.

Rename TPS22811 pin 2 to nEN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
Parts:
- D1: footprint EVO2513-0_5_0-import-fps:Diode DO-214AA SMB Not-Pol -> Diode_SMD:D_SMB
- LED1: footprint EVO2513-0_5_0-import-fps:LED 0603 H0-7 (C) -> LED_SMD:LED_0603_1608Metric
Changed lines of the file:
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@@
 			)
 		)
-		(property "Footprint" "EVO2513-0_5_0-import-fps:LED 0603 H0-7 (C)"
+		(property "Footprint" "LED_SMD:LED_0603_1608Metric"
 			(at 297.18 124.46 0)
 			(hide yes)
@@
 			)
 		)
-		(property "Footprint" "EVO2513-0_5_0-import-fps:Diode DO-214AA SMB Not-Pol"
+		(property "Footprint" "Diode_SMD:D_SMB"
 			(at 109.22 134.62 0)
 			(hide yes)

Commit message: Fill manufacturer part numbers from the 0.5.0 build orders
Set MANUFACTURER and MANUFACTURER_PN on every fitted part, in the
schematic and on the board. Unchanged parts take the exact part numbers
ordered for the 0.5.0 backup build (DigiKey list and Mouser basket);
changed parts reuse an ordered part where value, package and rating
match; the rest keep the schematic's part or take a Yageo RC/CC part.

Co-Authored-By: Claude Opus 5.5 <noreply@anthropic.com>
Parts:
- C1: MANUFACTURER (none) -> YAGEO; MANUFACTURER_PN (none) -> CC0402KRX7R9BB472
- D1: MANUFACTURER LittelFuse -> Littelfuse Inc.
- FL1: MANUFACTURER Murata -> Murata Electronics
- LED1: MANUFACTURER Everlight -> Everlight Electronics Co Ltd; MANUFACTURER_PN QTLP600C-4 -> QTLP600C4TR
- Q1, Q3: MANUFACTURER Diodes Inc -> Diodes Incorporated
- R1: MANUFACTURER (none) -> YAGEO; MANUFACTURER_PN (none) -> RC0402FR-07619KL
- R2: MANUFACTURER ? -> YAGEO; MANUFACTURER_PN ? -> RC0402FR-0712KL
- R3: MANUFACTURER ? -> YAGEO; MANUFACTURER_PN ? -> RC0402FR-07100KL
- R4, R5: MANUFACTURER (none) -> YAGEO; MANUFACTURER_PN (none) -> RC0402FR-0710RL
- R6: MANUFACTURER ? -> YAGEO; MANUFACTURER_PN ? -> RC0402FR-075K1L
- R7: MANUFACTURER ? -> YAGEO; MANUFACTURER_PN ? -> RC0402FR-0710KL
- U2: MANUFACTURER Analog Devices -> Analog Devices Inc.; MANUFACTURER_PN LTC4365IDDB -> LTC4365IDDB#TRPBF
Changed lines of the file:
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@@
 			)
 		)
-		(property "MANUFACTURER" "Murata"
+		(property "MANUFACTURER" "Murata Electronics"
 			(at 258.572 93.98 0)
 			(hide yes)
@@
 			)
 		)
-		(property "MANUFACTURER" ""
+		(property "MANUFACTURER" "YAGEO"
 			(at 124.714 148.082 0)
 			(hide yes)
@@
 			)
 		)
-		(property "MANUFACTURER_PN" ""
+		(property "MANUFACTURER_PN" "RC0402FR-07619KL"
 			(at 124.714 148.082 0)
 			(hide yes)
@@
 			)
 		)
-		(property "MANUFACTURER" ""
+		(property "MANUFACTURER" "YAGEO"
 			(at 197.612 171.45 0)
 			(hide yes)
@@
 			)
 		)
-		(property "MANUFACTURER_PN" ""
+		(property "MANUFACTURER_PN" "CC0402KRX7R9BB472"
 			(at 197.612 171.45 0)
 			(hide yes)
@@
 			)
 		)
-		(property "MANUFACTURER" "?"
+		(property "MANUFACTURER" "YAGEO"
 			(at 124.714 165.862 0)
 			(hide yes)
@@
 			)
 		)
-		(property "MANUFACTURER_PN" "?"
+		(property "MANUFACTURER_PN" "RC0402FR-0712KL"
 			(at 124.714 165.862 0)
 			(hide yes)
@@
 			)
 		)
-		(property "MANUFACTURER" ""
+		(property "MANUFACTURER" "YAGEO"
 			(at 200.914 125.222 0)
 			(hide yes)
@@
 			)
 		)
-		(property "MANUFACTURER_PN" ""
+		(property "MANUFACTURER_PN" "RC0402FR-0710RL"
 			(at 200.914 125.222 0)
 			(hide yes)
@@
 			)
 		)
-		(property "MANUFACTURER" "Analog Devices"
+		(property "MANUFACTURER" "Analog Devices Inc."
 			(at 173.482 144.78 0)
 			(hide yes)
@@
 			)
 		)
-		(property "MANUFACTURER_PN" "LTC4365IDDB"
+		(property "MANUFACTURER_PN" "LTC4365IDDB#TRPBF"
 			(at 173.482 144.78 0)
 			(hide yes)
@@
 			)
 		)
-		(property "MANUFACTURER" "Everlight"
+		(property "MANUFACTURER" "Everlight Electronics Co Ltd"
 			(at 295.91 120.142 90)
 			(hide yes)
@@
 			)
 		)
-		(property "MANUFACTURER_PN" "QTLP600C-4"
+		(property "MANUFACTURER_PN" "QTLP600C4TR"
 			(at 295.91 120.142 90)
 			(hide yes)
@@
 			)
 		)
-		(property "MANUFACTURER" "LittelFuse"
+		(property "MANUFACTURER" "Littelfuse Inc."
 			(at 107.95 130.302 90)
 			(hide yes)
@@
 			)
 		)
-		(property "MANUFACTURER" "Diodes Inc"
+		(property "MANUFACTURER" "Diodes Incorporated"
 			(at 206.502 93.98 0)
 			(hide yes)
@@
 			)
 		)
-		(property "MANUFACTURER" "?"
+		(property "MANUFACTURER" "YAGEO"
 			(at 296.164 107.442 0)
 			(hide yes)
@@
 			)
 		)
-		(property "MANUFACTURER_PN" "?"
+		(property "MANUFACTURER_PN" "RC0402FR-0710KL"
 			(at 296.164 107.442 0)
 			(hide yes)
@@
 			)
 		)
-		(property "MANUFACTURER" "?"
+		(property "MANUFACTURER" "YAGEO"
 			(at 200.914 159.512 0)
 			(hide yes)
@@
 			)
 		)
-		(property "MANUFACTURER_PN" "?"
+		(property "MANUFACTURER_PN" "RC0402FR-075K1L"
 			(at 200.914 159.512 0)
 			(hide yes)
@@
 			)
 		)
-		(property "MANUFACTURER" "?"
+		(property "MANUFACTURER" "YAGEO"
 			(at 139.954 140.462 0)
 			(hide yes)
@@
 			)
 		)
-		(property "MANUFACTURER_PN" "?"
+		(property "MANUFACTURER_PN" "RC0402FR-07100KL"
 			(at 139.954 140.462 0)
 			(hide yes)
@@
 			)
 		)
-		(property "MANUFACTURER" "Diodes Inc"
+		(property "MANUFACTURER" "Diodes Incorporated"
 			(at 179.832 93.98 0)
 			(hide yes)
@@
 			)
 		)
-		(property "MANUFACTURER" ""
+		(property "MANUFACTURER" "YAGEO"
 			(at 184.404 125.222 0)
 			(hide yes)
@@
 			)
 		)
-		(property "MANUFACTURER_PN" ""
+		(property "MANUFACTURER_PN" "RC0402FR-0710RL"
 			(at 184.404 125.222 0)
 			(hide yes)

Commit message: Match D1 and R14 to the parts held, standardise resistors on Yageo
D1 is the Diotec 1.0SMBJ26CA and R14 the Yageo PA2512FKE7W0R012E, as
received. R31 and R111-R114 move to Yageo so every resistor except the
current-sense shunts comes from one manufacturer.

Co-Authored-By: Claude Opus 5.5 <noreply@anthropic.com>
Parts:
- D1: value SMBJ26CA -> 1.0SMBJ26CA; ALTIUM_VALUE SMBJ26CA -> 1.0SMBJ26CA; MANUFACTURER Littelfuse Inc. -> Diotec Semiconductor; MANUFACTURER_PN SMBJ26CA -> 1.0SMBJ26CA
Changed lines of the file:
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@@
 			)
 		)
-		(property "Value" "SMBJ26CA"
+		(property "Value" "1.0SMBJ26CA"
 			(at 107.95 130.302 90)
 			(hide yes)
@@
 			)
 		)
-		(property "Description" "TVS SMBJ26CA 26V SMB"
+		(property "Description" "TVS 1.0SMBJ26CA 26V SMB"
 			(at 109.22 134.62 0)
 			(hide yes)
@@
 			)
 		)
-		(property "MANUFACTURER" "Littelfuse Inc."
+		(property "MANUFACTURER" "Diotec Semiconductor"
 			(at 107.95 130.302 90)
 			(hide yes)
@@
 			)
 		)
-		(property "MANUFACTURER_PN" "SMBJ26CA"
+		(property "MANUFACTURER_PN" "1.0SMBJ26CA"
 			(at 107.95 130.302 90)
 			(hide yes)
@@
 			)
 		)
-		(property "ALTIUM_VALUE" "SMBJ26CA"
+		(property "ALTIUM_VALUE" "1.0SMBJ26CA"
 			(at 110.49 136.906 90)
 			(show_name no)
