File: S04 Charger Regulation.kicad_sch (KiCad schematic)
At the start: 24 parts, among them Q6 DMT4011LFG, Q7 DMT4011LFG, U1 LTC1960

Commit message: Use KiCad standard footprints for chip resistors and capacitors
The imported Lattech R/C footprints have poor land patterns (the 0402s
use 0.635 mm circular pads) and cause tombstoning in assembly. Replace
all 139 chip resistors and capacitors with KiCad's standard IPC-7351
nominal footprints:

  Res 0402/0603/1206/2512 -> Resistor_SMD:R_xxxx_xxxxMetric (87)
  Cap 0402/0603/0805/1206/1210 -> Capacitor_SMD:C_xxxx_xxxxMetric (52)

Each part keeps its position, rotation, side, pad nets, schematic link
and reference/value text placement. The pads are on the same axis with
pad 1 on the same side, and every old pad centre lies inside the new
pad, so existing tracks still connect. Zones are refilled.

Schematic Footprint fields and the symbols' footprint filters point at
the new footprints, and the unused imported R/C footprints are removed
from the project library. Electrolytic capacitors are not changed.

DRC: 0 unconnected items, as before. Tracks, vias, zone outlines and
all other footprints are unchanged. 11 courtyard overlaps are new,
because the old footprints had no courtyards.

Co-Authored-By: Claude Opus 5.5 <noreply@anthropic.com>
Parts:
- C13, C14, C24, C25, C26: footprint EVO2513-0_5_0-import-fps:Cap 1206 H1-8 -> Capacitor_SMD:C_1206_3216Metric
- C15, C16: footprint EVO2513-0_5_0-import-fps:Cap 0805 H1-4 -> Capacitor_SMD:C_0805_2012Metric
- C17, C18, C19, C20, C21: footprint EVO2513-0_5_0-import-fps:Cap 0402 H0-6 R -> Capacitor_SMD:C_0402_1005Metric
- C22, C23: footprint EVO2513-0_5_0-import-fps:Cap 0603 H0-9 -> Capacitor_SMD:C_0603_1608Metric
- R19, R83: footprint EVO2513-0_5_0-import-fps:Res 2512 H0-9 -> Resistor_SMD:R_2512_6332Metric
- R20, R21: footprint EVO2513-0_5_0-import-fps:Res 0402 H0-45 R -> Resistor_SMD:R_0402_1005Metric
Changed lines of the file:
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@@
 			)
 		)
-		(property "Footprint" "EVO2513-0_5_0-import-fps:Cap 0402 H0-6 R"
+		(property "Footprint" "Capacitor_SMD:C_0402_1005Metric"
 			(at 222.25 180.1622 0)
 			(hide yes)
@@
 			)
 		)
-		(property "Footprint" "EVO2513-0_5_0-import-fps:Res 0402 H0-45 R"
+		(property "Footprint" "Resistor_SMD:R_0402_1005Metric"
 			(at 247.65 131.9022 0)
 			(hide yes)
@@
 			)
 		)
-		(property "Footprint" "EVO2513-0_5_0-import-fps:Cap 0805 H1-4"
+		(property "Footprint" "Capacitor_SMD:C_0805_2012Metric"
 			(at 149.86 172.5422 0)
 			(hide yes)
@@
 			)
 		)
-		(property "Footprint" "EVO2513-0_5_0-import-fps:Cap 1206 H1-8"
+		(property "Footprint" "Capacitor_SMD:C_1206_3216Metric"
 			(at 297.18 98.8822 0)
 			(hide yes)
@@
 			)
 		)
-		(property "Footprint" "EVO2513-0_5_0-import-fps:Cap 1206 H1-8"
+		(property "Footprint" "Capacitor_SMD:C_1206_3216Metric"
 			(at 77.47 97.6122 0)
 			(hide yes)
@@
 			)
 		)
-		(property "Footprint" "EVO2513-0_5_0-import-fps:Cap 0603 H0-9"
+		(property "Footprint" "Capacitor_SMD:C_0603_1608Metric"
 			(at 270.51 98.8822 0)
 			(hide yes)
@@
 			)
 		)
-		(property "Footprint" "EVO2513-0_5_0-import-fps:Cap 0402 H0-6 R"
+		(property "Footprint" "Capacitor_SMD:C_0402_1005Metric"
 			(at 247.65 144.6022 0)
 			(hide yes)
@@
 			)
 		)
-		(property "Footprint" "EVO2513-0_5_0-import-fps:Cap 1206 H1-8"
+		(property "Footprint" "Capacitor_SMD:C_1206_3216Metric"
 			(at 284.48 98.8822 0)
 			(hide yes)
@@
 			)
 		)
-		(property "Footprint" "EVO2513-0_5_0-import-fps:Res 0402 H0-45 R"
+		(property "Footprint" "Resistor_SMD:R_0402_1005Metric"
 			(at 232.41 170.0022 0)
 			(hide yes)
@@
 			)
 		)
-		(property "Footprint" "EVO2513-0_5_0-import-fps:Res 2512 H0-9"
+		(property "Footprint" "Resistor_SMD:R_2512_6332Metric"
 			(at 229.87 87.4522 0)
 			(hide yes)
@@
 			)
 		)
-		(property "Footprint" "EVO2513-0_5_0-import-fps:Cap 1206 H1-8"
+		(property "Footprint" "Capacitor_SMD:C_1206_3216Metric"
 			(at 309.88 98.8822 0)
 			(hide yes)
@@
 			)
 		)
-		(property "Footprint" "EVO2513-0_5_0-import-fps:Cap 0603 H0-9"
+		(property "Footprint" "Capacitor_SMD:C_0603_1608Metric"
 			(at 247.65 180.1622 0)
 			(hide yes)
@@
 			)
 		)
-		(property "Footprint" "EVO2513-0_5_0-import-fps:Cap 0402 H0-6 R"
+		(property "Footprint" "Capacitor_SMD:C_0402_1005Metric"
 			(at 160.02 172.5422 0)
 			(hide yes)
@@
 			)
 		)
-		(property "Footprint" "EVO2513-0_5_0-import-fps:Cap 0805 H1-4"
+		(property "Footprint" "Capacitor_SMD:C_0805_2012Metric"
 			(at 160.02 97.6122 0)
 			(hide yes)
@@
 			)
 		)
-		(property "Footprint" "EVO2513-0_5_0-import-fps:Cap 1206 H1-8"
+		(property "Footprint" "Capacitor_SMD:C_1206_3216Metric"
 			(at 88.9 97.6122 0)
 			(hide yes)
@@
 			)
 		)
-		(property "Footprint" "EVO2513-0_5_0-import-fps:Cap 0402 H0-6 R"
+		(property "Footprint" "Capacitor_SMD:C_0402_1005Metric"
 			(at 232.41 180.1622 0)
 			(hide yes)
@@
 			)
 		)
-		(property "Footprint" "EVO2513-0_5_0-import-fps:Res 2512 H0-9"
+		(property "Footprint" "Resistor_SMD:R_2512_6332Metric"
 			(at 229.87 82.3722 0)
 			(hide yes)
@@
 			)
 		)
-		(property "Footprint" "EVO2513-0_5_0-import-fps:Cap 0402 H0-6 R"
+		(property "Footprint" "Capacitor_SMD:C_0402_1005Metric"
 			(at 212.09 180.1622 0)
 			(hide yes)

Commit message: Fix schematic ERC issues from the import
ERC across all seven sheets reported 1481 issues from the import:

- Every item sat 43 mil off KiCad's 50 mil connection grid in Y, so new
  wires would not snap to existing pins. Each sheet's contents are
  shifted 7 mil (0.1778 mm) onto the grid; the library symbol
  definitions are untouched and a uniform shift keeps every connection.
  A few wire corners on S06 were off grid on their own (at 6740 mil,
  7620 mil and y 3290 mil); they move to the nearest grid point, which
  removes two 10 mil stubs and moves #PWR065 with its wire.
- Nine wires ran 1.27-2.54 mm past the label sitting on them (ID on S01;
  LDVR1/2 and HDVR1/2 on S06), leaving dangling ends. They are trimmed
  back to the label.
- GND, +12V, +3V3MCU and +5V enter through connector pins, so ERC had
  no power source for them. A PWR_FLAG (#FLG01-#FLG04) sits on each.
- The title-block module name used the Altium formula
  ${COPY(DOCUMENTNAME,5,LENGTH(DOCUMENTNAME)-11)}, which KiCad cannot
  evaluate. Each sheet now carries the title it produced.

ERC: 1481 -> 0. The netlist still matches the PCB's 147 nets.

Update PCB from Schematic was rerun afterwards. It changes metadata only:
footprint filters, unit and pin-function data from the symbols, and the
KiLib_Generator fields dropped from the 139 standard R/C footprints. No
placement or copper changes.

Co-Authored-By: Claude Opus 5.5 <noreply@anthropic.com>
Other:
- note added: "Charger Regulation"
- note removed: "${COPY(DOCUMENTNAME,5,LENGTH(DOCUMENTNAME)-11)}"

Commit message: Convert the schematic to a hierarchical root sheet
The Altium import produced seven KiCad 10 top-level sheets, with S01's
content in EVO2513-0_5_0.kicad_sch. kicad-cli only loads the first of
those, so command-line ERC, netlist and DRC parity checks saw S01 alone.

- EVO2513-0_5_0.kicad_sch is now a root sheet holding one sheet symbol per
  sheet; S01's content moves to "S01 External Connectors.kicad_sch".
- Each sheet symbol keeps its old top-level sheet UUID, so symbol
  references, net names and connectivity are unchanged: the netlist from
  the new root is identical to the previous whole-design netlist (229
  components, 147 nets). Cross-sheet nets still use global labels.
- The board's 229 footprint paths take the hierarchical form
  /<sheet>/<symbol>, and S01's footprints point at the new sheet file.
  No copper or placement changes.
- Every title block read "sheet 7 of 7" (a single DOCUMENTNUMBER project
  variable). Sheet numbers now use the page number: the root is page 1
  and S01-S07 are pages 2-8.

kicad-cli ERC over the whole design: 0 errors, 0 warnings. DRC with
schematic parity: 0 parity issues, 450 violations as before.

Co-Authored-By: Claude Opus 5.5 <noreply@anthropic.com>
Other:
- note added: "${#}"
- note removed: "${DOCUMENTNUMBER}"
Changed lines of the file:
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@@
 		)
 	)
-	(text "${DOCUMENTNUMBER}"
+	(text "${#}"
 		(exclude_from_sim no)
 		(at 298.45 292.1 0)
@@
 		(instances
 			(project "EVO2513-0_5_0"
-				(path "/18ff53f2-b256-4e35-9ef5-a5aab1ec179d"
+				(path "/44203427-0a3b-455b-9bb9-c1b577d179b3/18ff53f2-b256-4e35-9ef5-a5aab1ec179d"
 					(reference "#PWR055")
 					(unit 1)
@@
 		(instances
 			(project "EVO2513-0_5_0"
-				(path "/18ff53f2-b256-4e35-9ef5-a5aab1ec179d"
+				(path "/44203427-0a3b-455b-9bb9-c1b577d179b3/18ff53f2-b256-4e35-9ef5-a5aab1ec179d"
 					(reference "#PWR043")
 					(unit 1)
@@
 		(instances
 			(project "EVO2513-0_5_0"
-				(path "/18ff53f2-b256-4e35-9ef5-a5aab1ec179d"
+				(path "/44203427-0a3b-455b-9bb9-c1b577d179b3/18ff53f2-b256-4e35-9ef5-a5aab1ec179d"
 					(reference "C19")
 					(unit 1)
@@
 		(instances
 			(project "EVO2513-0_5_0"
-				(path "/18ff53f2-b256-4e35-9ef5-a5aab1ec179d"
+				(path "/44203427-0a3b-455b-9bb9-c1b577d179b3/18ff53f2-b256-4e35-9ef5-a5aab1ec179d"
 					(reference "#PWR042")
 					(unit 1)
@@
 		(instances
 			(project "EVO2513-0_5_0"
-				(path "/18ff53f2-b256-4e35-9ef5-a5aab1ec179d"
+				(path "/44203427-0a3b-455b-9bb9-c1b577d179b3/18ff53f2-b256-4e35-9ef5-a5aab1ec179d"
 					(reference "#PWR049")
 					(unit 1)
@@
 		(instances
 			(project "EVO2513-0_5_0"
-				(path "/18ff53f2-b256-4e35-9ef5-a5aab1ec179d"
+				(path "/44203427-0a3b-455b-9bb9-c1b577d179b3/18ff53f2-b256-4e35-9ef5-a5aab1ec179d"
 					(reference "#PWR052")
 					(unit 1)
@@
 		(instances
 			(project "EVO2513-0_5_0"
-				(path "/18ff53f2-b256-4e35-9ef5-a5aab1ec179d"
+				(path "/44203427-0a3b-455b-9bb9-c1b577d179b3/18ff53f2-b256-4e35-9ef5-a5aab1ec179d"
 					(reference "R21")
 					(unit 1)
@@
 		(instances
 			(project "EVO2513-0_5_0"
-				(path "/18ff53f2-b256-4e35-9ef5-a5aab1ec179d"
+				(path "/44203427-0a3b-455b-9bb9-c1b577d179b3/18ff53f2-b256-4e35-9ef5-a5aab1ec179d"
 					(reference "#PWR045")
 					(unit 1)
@@
 		(instances
 			(project "EVO2513-0_5_0"
-				(path "/18ff53f2-b256-4e35-9ef5-a5aab1ec179d"
+				(path "/44203427-0a3b-455b-9bb9-c1b577d179b3/18ff53f2-b256-4e35-9ef5-a5aab1ec179d"
 					(reference "C15")
 					(unit 1)
@@
 		(instances
 			(project "EVO2513-0_5_0"
-				(path "/18ff53f2-b256-4e35-9ef5-a5aab1ec179d"
+				(path "/44203427-0a3b-455b-9bb9-c1b577d179b3/18ff53f2-b256-4e35-9ef5-a5aab1ec179d"
 					(reference "#PWR041")
 					(unit 1)
@@
 		(instances
 			(project "EVO2513-0_5_0"
-				(path "/18ff53f2-b256-4e35-9ef5-a5aab1ec179d"
+				(path "/44203427-0a3b-455b-9bb9-c1b577d179b3/18ff53f2-b256-4e35-9ef5-a5aab1ec179d"
 					(reference "#PWR048")
 					(unit 1)
@@
 		(instances
 			(project "EVO2513-0_5_0"
-				(path "/18ff53f2-b256-4e35-9ef5-a5aab1ec179d"
+				(path "/44203427-0a3b-455b-9bb9-c1b577d179b3/18ff53f2-b256-4e35-9ef5-a5aab1ec179d"
 					(reference "Q6")
 					(unit 1)
@@
 		(instances
 			(project "EVO2513-0_5_0"
-				(path "/18ff53f2-b256-4e35-9ef5-a5aab1ec179d"
+				(path "/44203427-0a3b-455b-9bb9-c1b577d179b3/18ff53f2-b256-4e35-9ef5-a5aab1ec179d"
 					(reference "#PWR046")
 					(unit 1)
@@
 		(instances
 			(project "EVO2513-0_5_0"
-				(path "/18ff53f2-b256-4e35-9ef5-a5aab1ec179d"
+				(path "/44203427-0a3b-455b-9bb9-c1b577d179b3/18ff53f2-b256-4e35-9ef5-a5aab1ec179d"
 					(reference "L1")
 					(unit 1)
@@
 		(instances
 			(project "EVO2513-0_5_0"
-				(path "/18ff53f2-b256-4e35-9ef5-a5aab1ec179d"
+				(path "/44203427-0a3b-455b-9bb9-c1b577d179b3/18ff53f2-b256-4e35-9ef5-a5aab1ec179d"
 					(reference "C25")
 					(unit 1)
@@
 		(instances
 			(project "EVO2513-0_5_0"
-				(path "/18ff53f2-b256-4e35-9ef5-a5aab1ec179d"
+				(path "/44203427-0a3b-455b-9bb9-c1b577d179b3/18ff53f2-b256-4e35-9ef5-a5aab1ec179d"
 					(reference "C13")
 					(unit 1)
@@
 		(instances
 			(project "EVO2513-0_5_0"
-				(path "/18ff53f2-b256-4e35-9ef5-a5aab1ec179d"
+				(path "/44203427-0a3b-455b-9bb9-c1b577d179b3/18ff53f2-b256-4e35-9ef5-a5aab1ec179d"
 					(reference "#PWR044")
 					(unit 1)
@@
 		(instances
 			(project "EVO2513-0_5_0"
-				(path "/18ff53f2-b256-4e35-9ef5-a5aab1ec179d"
+				(path "/44203427-0a3b-455b-9bb9-c1b577d179b3/18ff53f2-b256-4e35-9ef5-a5aab1ec179d"
 					(reference "C23")
 					(unit 1)
@@
 		(instances
 			(project "EVO2513-0_5_0"
-				(path "/18ff53f2-b256-4e35-9ef5-a5aab1ec179d"
+				(path "/44203427-0a3b-455b-9bb9-c1b577d179b3/18ff53f2-b256-4e35-9ef5-a5aab1ec179d"
 					(reference "#PWR040")
 					(unit 1)
@@
 		(instances
 			(project "EVO2513-0_5_0"
-				(path "/18ff53f2-b256-4e35-9ef5-a5aab1ec179d"
+				(path "/44203427-0a3b-455b-9bb9-c1b577d179b3/18ff53f2-b256-4e35-9ef5-a5aab1ec179d"
 					(reference "C21")
 					(unit 1)
@@
 		(instances
 			(project "EVO2513-0_5_0"
-				(path "/18ff53f2-b256-4e35-9ef5-a5aab1ec179d"
+				(path "/44203427-0a3b-455b-9bb9-c1b577d179b3/18ff53f2-b256-4e35-9ef5-a5aab1ec179d"
 					(reference "Q7")
 					(unit 1)
@@
 		(instances
 			(project "EVO2513-0_5_0"
-				(path "/18ff53f2-b256-4e35-9ef5-a5aab1ec179d"
+				(path "/44203427-0a3b-455b-9bb9-c1b577d179b3/18ff53f2-b256-4e35-9ef5-a5aab1ec179d"
 					(reference "#PWR053")
 					(unit 1)
@@
 		(instances
 			(project "EVO2513-0_5_0"
-				(path "/18ff53f2-b256-4e35-9ef5-a5aab1ec179d"
+				(path "/44203427-0a3b-455b-9bb9-c1b577d179b3/18ff53f2-b256-4e35-9ef5-a5aab1ec179d"
 					(reference "C24")
 					(unit 1)
@@
 		(instances
 			(project "EVO2513-0_5_0"
-				(path "/18ff53f2-b256-4e35-9ef5-a5aab1ec179d"
+				(path "/44203427-0a3b-455b-9bb9-c1b577d179b3/18ff53f2-b256-4e35-9ef5-a5aab1ec179d"
 					(reference "R20")
 					(unit 1)
@@
 		(instances
 			(project "EVO2513-0_5_0"
-				(path "/18ff53f2-b256-4e35-9ef5-a5aab1ec179d"
+				(path "/44203427-0a3b-455b-9bb9-c1b577d179b3/18ff53f2-b256-4e35-9ef5-a5aab1ec179d"
 					(reference "#PWR051")
 					(unit 1)
@@
 		(instances
 			(project "EVO2513-0_5_0"
-				(path "/18ff53f2-b256-4e35-9ef5-a5aab1ec179d"
+				(path "/44203427-0a3b-455b-9bb9-c1b577d179b3/18ff53f2-b256-4e35-9ef5-a5aab1ec179d"
 					(reference "U1")
 					(unit 2)
@@
 		(instances
 			(project "EVO2513-0_5_0"
-				(path "/18ff53f2-b256-4e35-9ef5-a5aab1ec179d"
+				(path "/44203427-0a3b-455b-9bb9-c1b577d179b3/18ff53f2-b256-4e35-9ef5-a5aab1ec179d"
 					(reference "R19")
 					(unit 1)
@@
 		(instances
 			(project "EVO2513-0_5_0"
-				(path "/18ff53f2-b256-4e35-9ef5-a5aab1ec179d"
+				(path "/44203427-0a3b-455b-9bb9-c1b577d179b3/18ff53f2-b256-4e35-9ef5-a5aab1ec179d"
 					(reference "C26")
 					(unit 1)
@@
 		(instances
 			(project "EVO2513-0_5_0"
-				(path "/18ff53f2-b256-4e35-9ef5-a5aab1ec179d"
+				(path "/44203427-0a3b-455b-9bb9-c1b577d179b3/18ff53f2-b256-4e35-9ef5-a5aab1ec179d"
 					(reference "C22")
 					(unit 1)
@@
 		(instances
 			(project "EVO2513-0_5_0"
-				(path "/18ff53f2-b256-4e35-9ef5-a5aab1ec179d"
+				(path "/44203427-0a3b-455b-9bb9-c1b577d179b3/18ff53f2-b256-4e35-9ef5-a5aab1ec179d"
 					(reference "#PWR047")
 					(unit 1)
@@
 		(instances
 			(project "EVO2513-0_5_0"
-				(path "/18ff53f2-b256-4e35-9ef5-a5aab1ec179d"
+				(path "/44203427-0a3b-455b-9bb9-c1b577d179b3/18ff53f2-b256-4e35-9ef5-a5aab1ec179d"
 					(reference "C17")
 					(unit 1)
@@
 		(instances
 			(project "EVO2513-0_5_0"
-				(path "/18ff53f2-b256-4e35-9ef5-a5aab1ec179d"
+				(path "/44203427-0a3b-455b-9bb9-c1b577d179b3/18ff53f2-b256-4e35-9ef5-a5aab1ec179d"
 					(reference "#PWR054")
 					(unit 1)
@@
 		(instances
 			(project "EVO2513-0_5_0"
-				(path "/18ff53f2-b256-4e35-9ef5-a5aab1ec179d"
+				(path "/44203427-0a3b-455b-9bb9-c1b577d179b3/18ff53f2-b256-4e35-9ef5-a5aab1ec179d"
 					(reference "D2")
 					(unit 1)
@@
 		(instances
 			(project "EVO2513-0_5_0"
-				(path "/18ff53f2-b256-4e35-9ef5-a5aab1ec179d"
+				(path "/44203427-0a3b-455b-9bb9-c1b577d179b3/18ff53f2-b256-4e35-9ef5-a5aab1ec179d"
 					(reference "C16")
 					(unit 1)
@@
 		(instances
 			(project "EVO2513-0_5_0"
-				(path "/18ff53f2-b256-4e35-9ef5-a5aab1ec179d"
+				(path "/44203427-0a3b-455b-9bb9-c1b577d179b3/18ff53f2-b256-4e35-9ef5-a5aab1ec179d"
 					(reference "C14")
 					(unit 1)
@@
 		(instances
 			(project "EVO2513-0_5_0"
-				(path "/18ff53f2-b256-4e35-9ef5-a5aab1ec179d"
+				(path "/44203427-0a3b-455b-9bb9-c1b577d179b3/18ff53f2-b256-4e35-9ef5-a5aab1ec179d"
 					(reference "C20")
 					(unit 1)
@@
 		(instances
 			(project "EVO2513-0_5_0"
-				(path "/18ff53f2-b256-4e35-9ef5-a5aab1ec179d"
+				(path "/44203427-0a3b-455b-9bb9-c1b577d179b3/18ff53f2-b256-4e35-9ef5-a5aab1ec179d"
 					(reference "#PWR039")
 					(unit 1)
@@
 		(instances
 			(project "EVO2513-0_5_0"
-				(path "/18ff53f2-b256-4e35-9ef5-a5aab1ec179d"
+				(path "/44203427-0a3b-455b-9bb9-c1b577d179b3/18ff53f2-b256-4e35-9ef5-a5aab1ec179d"
 					(reference "R83")
 					(unit 1)
@@
 		(instances
 			(project "EVO2513-0_5_0"
-				(path "/18ff53f2-b256-4e35-9ef5-a5aab1ec179d"
+				(path "/44203427-0a3b-455b-9bb9-c1b577d179b3/18ff53f2-b256-4e35-9ef5-a5aab1ec179d"
 					(reference "D3")
 					(unit 1)
@@
 		(instances
 			(project "EVO2513-0_5_0"
-				(path "/18ff53f2-b256-4e35-9ef5-a5aab1ec179d"
+				(path "/44203427-0a3b-455b-9bb9-c1b577d179b3/18ff53f2-b256-4e35-9ef5-a5aab1ec179d"
 					(reference "C18")
 					(unit 1)
@@
 		(instances
 			(project "EVO2513-0_5_0"
-				(path "/18ff53f2-b256-4e35-9ef5-a5aab1ec179d"
+				(path "/44203427-0a3b-455b-9bb9-c1b577d179b3/18ff53f2-b256-4e35-9ef5-a5aab1ec179d"
 					(reference "#PWR050")
 					(unit 1)
@@
 		(instances
 			(project "EVO2513-0_5_0"
-				(path "/18ff53f2-b256-4e35-9ef5-a5aab1ec179d"
+				(path "/44203427-0a3b-455b-9bb9-c1b577d179b3/18ff53f2-b256-4e35-9ef5-a5aab1ec179d"
 					(reference "#FLG04")
 					(unit 1)
@@
 		)
 	)
-	(sheet_instances
-		(path "/"
-			(page "4")
-		)
-	)

Commit message: Link the sheets through hierarchical labels and sheet pins
The 78 cross-sheet global labels on S01-S07 become hierarchical labels,
and each sheet symbol on the root gets a pin per label name (71 pins).
On the root, each pin connects through a short wire to a global label
with the net name. Global labels there, rather than local ones, keep the
35 net names free of a "/" sheet-path prefix, so the net classes and the
board's nets are unchanged.

Layout: S01 External Connectors on the left with its pins on the right
edge; S02-S04 and S05-S07 in two columns with their pins on the left.

The netlist is identical to before (229 components, 147 nets, same names
and pins). kicad-cli ERC: 0 errors, 0 warnings. DRC with schematic
parity: 0 parity issues, 450 violations as before.

Co-Authored-By: Claude Opus 5.5 <noreply@anthropic.com>
Changed lines of the file:
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@@
 		)
 	)
-	(global_label "DCCHARGER"
+	(hierarchical_label "DCCHARGER"
 		(shape passive)
 		(at 334.01 87.63 0)
-		(fields_autoplaced yes)
 		(effects
 			(font
@@
 			(justify left)
 		)
-		(property "Intersheetrefs" "${INTERSHEET_REFS}"
-			(at 334.01 87.63 0)
-			(effects
-				(font
-					(size 1.27 1.27)
-				)
-				(justify left)
-				(hide yes)
-			)
-		)
 	)
-	(global_label "DCSENSED"
+	(hierarchical_label "DCSENSED"
 		(shape passive)
 		(at 53.34 87.63 180)
-		(fields_autoplaced yes)
 		(effects
 			(font
@@
 			(justify right)
 		)
-		(property "Intersheetrefs" "${INTERSHEET_REFS}"
-			(at 53.34 87.63 0)
-			(effects
-				(font
-					(size 1.27 1.27)
-				)
-				(justify right)
-				(hide yes)
-			)
-		)
 	)
