File: EVO2513-0_5_0.kicad_pcb (KiCad board)
At the start: 8 copper layers, 110 x 69 mm, 256 parts, among them J1 1053101204, J2 1053101114, J3 10144517-043802LF, J4 1053102204, J5 1053091102, J6 1053091102, M1 78614150960, M2 78614150960, M3 78614150960, M4 78614150960, M5 78614150960, M6 78614150960, Q1 DMT6007LFGQ-7, Q10 DMT4011LFG, Q11 DMT4011LFG, Q12 DMP3018SFV, Q13 DMP3018SFV, Q14 DMP3018SFV, Q15 DMP3018SFV, Q16 IAUCN04S7L019, Q17 IAUCN04S7L028, Q18 CSD17304Q3, Q19 IAUCN04S7L019, Q20 BSS138, Q21 BSS138, Q22 BSS138, Q23 BSS138, Q3 DMT6007LFGQ-7, Q4 DMP3018SFV, Q5 DMP3018SFV, Q6 DMT4011LFG, Q7 DMT4011LFG, Q8 DMT4011LFG, Q9 DMT4011LFG, U1 LTC1960, U10 TLV9002IDSG, U11 PCAL9714, U2 LTC4365, U5 LM51772RHAR, U6 TPS22811, U7 TPS22811, U8 TLV9002IDSG, U9 TPS22811

Commit message: Final-revision value changes and standard R/C symbols
Values (schematic and PCB):
- C2 100uF -> 82uF, matching the ordered 35SVPF82M
- C46, C47, C51 (TPS22811 DVDT) 4.7nF -> 1.8nF CC0402KRX7R9BB182 for a
  shorter output ramp
- R24-R27 10R -> 0R; D9, D10 and R36 DNP
- R14 0.01R -> 0.012R PA2512FKF7W0R012E

Symbols:
- All 160 resistors and capacitors now use Device:R, Device:C and
  Device:C_Polarized; the 76 per-value R/C symbols are removed from the
  project library. Connectivity is unchanged (netlist compared).
- Value is now the displayed field instead of ALTIUM_VALUE, which had left
  R1, C39 and R54 showing their old values. ALTIUM_VALUE synced with Value
  on R1, C39, R54, D1, Q1, Q3 and L1.
- Net-(C40-+) is now Net-(U5-ISNSP); renamed on the PCB and in the
  PWR 15A net class pattern.

Co-Authored-By: Claude Opus 5.5 <noreply@anthropic.com>
Parts:
- C2: value 100uF -> 82uF
- C46, C47, C51: value 4.7nF -> 1.8nF
- R14: value 0.01R -> 0.012R
- R24, R25, R26, R27: value 10R -> 0R
