File: EVO2513-0_5_0.kicad_pcb (KiCad board)
At the start: 8 copper layers, 110 x 69 mm, 256 parts, among them J1 1053101204, J2 1053101114, J3 10144517-043802LF, J4 1053102204, J5 1053091102, J6 1053091102, M1 78614150960, M2 78614150960, M3 78614150960, M4 78614150960, M5 78614150960, M6 78614150960, Q1 DMT6007LFGQ-7, Q10 DMT4011LFG, Q11 DMT4011LFG, Q12 DMP3018SFV, Q13 DMP3018SFV, Q14 DMP3018SFV, Q15 DMP3018SFV, Q16 IAUCN04S7L019, Q17 IAUCN04S7L028, Q18 CSD17304Q3, Q19 IAUCN04S7L019, Q20 BSS138, Q21 BSS138, Q22 BSS138, Q23 BSS138, Q3 DMT6007LFGQ-7, Q4 DMP3018SFV, Q5 DMP3018SFV, Q6 DMT4011LFG, Q7 DMT4011LFG, Q8 DMT4011LFG, Q9 DMT4011LFG, U1 LTC1960, U10 TLV9002IDSG, U11 PCAL9714, U2 LTC4365, U5 LM51772RHAR, U6 TPS22811, U7 TPS22811, U8 TLV9002IDSG, U9 TPS22811

Commit message: Retune load-switch OVLO and PG dividers; add design constraint notes
- R90-R92 1M -> 1.07M: OVLO trips at 14.0 V (13.40-14.69 V) and recovers
  below 12.75 V (at least 12.23 V), so a tripped switch always comes back
  on the 12.03 V rail. R101 (Q23 gate divider) -> 1.07M to share the line.
- PGTH dividers R59/R61/R76 1M -> 100K and R60/R62/R77 130K -> 13K: same
  10.43 V threshold, but the +-1 uA pin leakage now moves it 0.1 V, not
  1 V; worst-case rising 10.93 V instead of 11.84 V.
- Schematic notes for the W16 constraints: J2 contacts (S01), R16 latching
  breaker and ED29/QE29 trip currents (S03), R19 vs L1 saturation (S04),
  R22 presence pull-up (S05), R42 and the U5 MODE/ILIMCOMP/VCC2 pins (S06),
  and the OVLO/PG divider settings (S07).
- README: OVLO and PG divider figures, and the EN_CONST_TDEAD default for
  the I2C build.

Co-Authored-By: Claude Opus 5.5 <noreply@anthropic.com>
Parts:
- R101, R90, R91, R92: value 1M -> 1.07M
- R59, R61, R76: value 1M -> 100K
- R60, R62, R77: value 130K -> 13K
Changed lines of the file:
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@@
 			)
 		)
-		(property "Value" "130K"
+		(property "Value" "13K"
 			(at 123.6738 -299.643043 0)
 			(unlocked yes)
@@
 			)
 		)
-		(property "Description" "Resistor 130K 1% 0402"
+		(property "Description" "Resistor 13K 1% 0402"
 			(at 0 0 270)
 			(layer "F.Fab")
@@
 			)
 		)
-		(property "ALTIUM_VALUE" "130K"
+		(property "ALTIUM_VALUE" "13K"
 			(at 0 0 270)
 			(unlocked yes)
@@
 			)
 		)
-		(property "Value" "1M"
+		(property "Value" "1.07M"
 			(at 0 1.17 0)
 			(layer "F.Fab")
@@
 			)
 		)
-		(property "Description" "Resistor 1M 1% 0402"
+		(property "Description" "Resistor 1.07M 1% 0402"
 			(at 0 0 0)
 			(layer "F.Fab")
@@
 			)
 		)
-		(property "ALTIUM_VALUE" "1M"
+		(property "ALTIUM_VALUE" "1.07M"
 			(at 0 0 0)
 			(unlocked yes)
@@
 			)
 		)
-		(property "Value" "130K"
+		(property "Value" "13K"
 			(at 123.6738 -299.643043 0)
 			(unlocked yes)
@@
 			)
 		)
-		(property "Description" "Resistor 130K 1% 0402"
+		(property "Description" "Resistor 13K 1% 0402"
 			(at 0 0 270)
 			(layer "F.Fab")
@@
 			)
 		)
-		(property "ALTIUM_VALUE" "130K"
+		(property "ALTIUM_VALUE" "13K"
 			(at 0 0 270)
 			(unlocked yes)
@@
 			)
 		)
-		(property "Value" "130K"
+		(property "Value" "13K"
 			(at 123.6738 -299.643043 0)
 			(unlocked yes)
@@
 			)
 		)
-		(property "Description" "Resistor 130K 1% 0402"
+		(property "Description" "Resistor 13K 1% 0402"
 			(at 0 0 270)
 			(layer "F.Fab")
@@
 			)
 		)
-		(property "ALTIUM_VALUE" "130K"
+		(property "ALTIUM_VALUE" "13K"
 			(at 0 0 270)
 			(unlocked yes)
@@
 			)
 		)
-		(property "Value" "1M"
+		(property "Value" "100K"
 			(at -123.6738 299.724071 0)
 			(unlocked yes)
@@
 			)
 		)
-		(property "Description" "Resistor 1M 1% 0402"
+		(property "Description" "Resistor 100K 1% 0402"
 			(at 0 0 90)
 			(layer "F.Fab")
@@
 			)
 		)
-		(property "ALTIUM_VALUE" "1M"
+		(property "ALTIUM_VALUE" "100K"
 			(at 0 0 90)
 			(unlocked yes)
@@
 			)
 		)
-		(property "Value" "1M"
+		(property "Value" "100K"
 			(at -123.6738 299.724071 0)
 			(unlocked yes)
@@
 			)
 		)
-		(property "Description" "Resistor 1M 1% 0402"
+		(property "Description" "Resistor 100K 1% 0402"
 			(at 0 0 90)
 			(layer "F.Fab")
@@
 			)
 		)
-		(property "ALTIUM_VALUE" "1M"
+		(property "ALTIUM_VALUE" "100K"
 			(at 0 0 90)
 			(unlocked yes)
@@
 			)
 		)
-		(property "Value" "1M"
+		(property "Value" "1.07M"
 			(at 0 1.17 0)
 			(layer "F.Fab")
@@
 			)
 		)
-		(property "Description" "Resistor 1M 1% 0402"
+		(property "Description" "Resistor 1.07M 1% 0402"
 			(at 0 0 0)
 			(layer "F.Fab")
@@
 			)
 		)
-		(property "ALTIUM_VALUE" "1M"
+		(property "ALTIUM_VALUE" "1.07M"
 			(at 0 0 0)
 			(unlocked yes)
@@
 			)
 		)
-		(property "Value" "1M"
+		(property "Value" "1.07M"
 			(at 0 1.17 0)
 			(layer "F.Fab")
@@
 			)
 		)
-		(property "Description" "Resistor 1M 1% 0402"
+		(property "Description" "Resistor 1.07M 1% 0402"
 			(at 0 0 0)
 			(layer "F.Fab")
@@
 			)
 		)
-		(property "ALTIUM_VALUE" "1M"
+		(property "ALTIUM_VALUE" "1.07M"
 			(at 0 0 0)
 			(unlocked yes)
@@
 			)
 		)
-		(property "Value" "1M"
+		(property "Value" "1.07M"
 			(at 0 1.17 0)
 			(layer "F.Fab")
@@
 			)
 		)
-		(property "Description" "Resistor 1M 1% 0402"
+		(property "Description" "Resistor 1.07M 1% 0402"
 			(at 0 0 0)
 			(layer "F.Fab")
@@
 			)
 		)
-		(property "ALTIUM_VALUE" "1M"
+		(property "ALTIUM_VALUE" "1.07M"
 			(at 0 0 0)
 			(unlocked yes)
@@
 			)
 		)
-		(property "Value" "1M"
+		(property "Value" "100K"
 			(at -123.6738 299.724071 0)
 			(unlocked yes)
@@
 			)
 		)
-		(property "Description" "Resistor 1M 1% 0402"
+		(property "Description" "Resistor 100K 1% 0402"
 			(at 0 0 90)
 			(layer "F.Fab")
@@
 			)
 		)
-		(property "ALTIUM_VALUE" "1M"
+		(property "ALTIUM_VALUE" "100K"
 			(at 0 0 90)
 			(unlocked yes)
