File: S06 STEP-Up Step-Down Reg.kicad_sch (KiCad schematic)
At the start: 53 parts, among them Q16 IAUCN04S7L019, Q17 IAUCN04S7L028, Q18 CSD17304Q3, Q19 IAUCN04S7L019, U5 LM51772RHAR

Commit message: WIP gate resistors
Parts:
- added R111, R112, R113, R114: 3R, Resistor_SMD:R_0603_1608Metric, symbol Device:R
Connections:
- net HDVR1: now also R111.2; no longer Q16.4 (G)
- net HDVR2: now also R113.1; no longer Q18.4 (G)
- net LDVR1: now also R112.1; no longer Q17.4 (G)
- net LDVR2: now also R114.2; no longer Q19.4 (G)
- new net: Q17.4 (G), R112.2
- new net: Q19.4 (G), R114.1
- new net: Q16.4 (G), R111.1
- new net: Q18.4 (G), R113.2
