File: S05 Battery Management.kicad_sch (KiCad schematic)
At the start: 17 parts, among them Q10 DMT4011LFG, Q11 DMT4011LFG, Q12 DMP3007SCG-13, Q13 DMP3007SCG-13, Q14 DMP3007SCG-13, Q15 DMP3007SCG-13, Q8 DMT4011LFG, Q9 DMT4011LFG, U1 LTC1960

Commit message: Keep top copper out of power FET source-drain gaps; mask-layer logo
- Add F.Cu keepouts (no tracks/vias/pour) between source and drain pads
  in the TDSON, CSD17304Q3 and PowerDI3333 footprints, so a shorted FET
  can be reworked without bridging S-D through top copper.
- Add Diodes_PowerDI3333-8 (copy of the KiCad Package_SON footprint with
  the keepout) and point Q4/Q5/Q12-Q15 at it; drop the board-level
  Q5/Q7 keepouts.
- Move nine vias (Q17 GND, Q18 SW2) out of the S-D gaps.
- New dru rule "Power FET pad to pour": 0.3 mm zone-to-pad clearance on
  Q footprints, giving >=0.25 mm mask web around FET pads.
- Add EVOSONIC_DNA_LOGO_390X600_MASK footprint (F.Mask polygons) and
  use it for LOGO01.
- Schematic NOTE fields updated and pushed to the PCB; zones refilled.
- README notes on the keepouts and the 0.3 mm rule.

ERC 0 violations. DRC 0 unconnected, 0 parity; remaining items are
excluded layer-marker edge clearances, silk overlap and text thickness.

Co-Authored-By: Claude Opus 5.5 <noreply@anthropic.com>
Parts:
- Q12, Q13, Q14, Q15: footprint Package_SON:Diodes_PowerDI3333-8 -> EVO2513-0_5_0-import-fps:Diodes_PowerDI3333-8
Changed lines of the file:
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@@
 			)
 		)
-		(property "Footprint" "Package_SON:Diodes_PowerDI3333-8"
+		(property "Footprint" "EVO2513-0_5_0-import-fps:Diodes_PowerDI3333-8"
 			(at 181.61 151.13 0)
 			(hide yes)
@@
 			)
 		)
-		(property "Footprint" "Package_SON:Diodes_PowerDI3333-8"
+		(property "Footprint" "EVO2513-0_5_0-import-fps:Diodes_PowerDI3333-8"
 			(at 193.04 59.69 0)
 			(hide yes)
@@
 			)
 		)
-		(property "Footprint" "Package_SON:Diodes_PowerDI3333-8"
+		(property "Footprint" "EVO2513-0_5_0-import-fps:Diodes_PowerDI3333-8"
 			(at 182.88 59.69 0)
 			(hide yes)
@@
 			)
 		)
-		(property "Footprint" "Package_SON:Diodes_PowerDI3333-8"
+		(property "Footprint" "EVO2513-0_5_0-import-fps:Diodes_PowerDI3333-8"
 			(at 191.77 151.13 0)
 			(hide yes)

Commit message: Raise divider impedances, dim the PG LEDs, use standard diode lands
TI asks for a pull-up of at least 350 kOhm on EN/UVLO above 5 V.
R108 100K -> 619K and R49 12K -> 75K, both values already on the
BOM: turn-on 11.10 V (10.63-11.91 V worst case), off 10.09 V. 1M/120K
was rejected because leakage across 1M puts worst-case turn-on at
12.24 V, above the rail.

Q24 gate bias R109 100K -> 1.07M and R110 27K -> 390K: +12V draw
94 -> 8.2 uA, gate 3.2 V at 12 V and under 4 V worst case at the
14.7 V OVLO limit. The R115 bypass pull-down is now 62.9K.

PGTH dividers R59/R61/R76 100K -> 390K and R60/R62/R77 13K -> 51K:
PG at 10.38 V (11.17 V worst case), 23.5 uA at threshold to meet TI's
20x PGTH leakage rule. 390K is the only new BOM value.

PG LED resistors R67/R68/R81 2.2K -> 4.7K, about 0.9 mA less on
battery with all rails up.

D1, D4, D6-D10 and LED1-LED4 move from imported Altium lands to KiCad
standard footprints (D_SMB, D_SMA, SOT-23, Diodes_UDFN-10, LED_0603),
in place with the same nets; the LEDs turn 180 deg for pad 1. Drops
the 8 thin LED A/C silk warnings. Five unused imported footprints
removed. Nearby parts and tracks adjusted for the new lands.

Keep the GND planes free of power copper, as on the original: remove
the SW1/L2 and SW2 strip zones and the small +12V (via block by R115)
and U5 ISNSP (under Q18's drain) zones from In1/In3/In5/In6. They
carried no current; GND gains about 0.8 mm2 on In1, 3.5 mm2 on In3
and In5 and 3.7 mm2 on In6 under the power stage.

Remove the 347 via-block octagons the Altium import left as copper
graphic polygons (gr_poly) on B.Cu and In1-In6, one 1.2 x 1.8 mm
octagon per six-via block per layer. As drawings they bypassed zone
rules, and on the GND layers they were net islands in the pour,
including the charger switch node. None carried current: same-net
pours connect the vias solid, and DRC finds 0 unconnected. GND gains
about 26 mm2 on In1, 21 mm2 on In3 and In5, 18 mm2 on In6 and 27 mm2
on B.Cu.

Rename TPS22811 pin 2 to nEN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
Parts:
- D10, D9: footprint EVO2513-0_5_0-import-fps:U-DFN2510-10 DIODE INC -> Package_DFN_QFN:Diodes_UDFN-10_1x2.5mm_P0.5mm
- D4: footprint EVO2513-0_5_0-import-fps:SOT-23 3-Pin -> Package_TO_SOT_SMD:SOT-23
Other:
- note added: "R22 = 1K is the D4 battery-presence pull-up: an empty battery slot sits at about 5 V. Expected. Keep R22 at 1K"
- note removed: "R22 = 1K is the D4 battery-presence pull-up: an empty battery slot sits at about 5 V. Expected. Keep R22 at 1K (R54 is 768R; they don't share a value)."
Changed lines of the file:
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@@
 		)
 	)
-	(text "R22 = 1K is the D4 battery-presence pull-up:\nan empty battery slot sits at about 5 V. Expected.\nKeep R22 at 1K (R54 is 768R; they don't share a value)."
+	(text "R22 = 1K is the D4 battery-presence pull-up:\nan empty battery slot sits at about 5 V. Expected.\nKeep R22 at 1K"
 		(exclude_from_sim no)
 		(at 68.58 116.84 0)
@@
 			)
 		)
-		(property "Footprint" "EVO2513-0_5_0-import-fps:U-DFN2510-10 DIODE INC"
+		(property "Footprint" "Package_DFN_QFN:Diodes_UDFN-10_1x2.5mm_P0.5mm"
 			(at 323.85 176.53 0)
 			(hide yes)
@@
 			)
 		)
-		(property "Footprint" "EVO2513-0_5_0-import-fps:U-DFN2510-10 DIODE INC"
+		(property "Footprint" "Package_DFN_QFN:Diodes_UDFN-10_1x2.5mm_P0.5mm"
 			(at 323.85 81.28 0)
 			(hide yes)
@@
 			)
 		)
-		(property "Footprint" "EVO2513-0_5_0-import-fps:SOT-23 3-Pin"
+		(property "Footprint" "Package_TO_SOT_SMD:SOT-23"
 			(at 52.07 123.19 0)
 			(hide yes)

Commit message: Fill manufacturer part numbers from the 0.5.0 build orders
Set MANUFACTURER and MANUFACTURER_PN on every fitted part, in the
schematic and on the board. Unchanged parts take the exact part numbers
ordered for the 0.5.0 backup build (DigiKey list and Mouser basket);
changed parts reuse an ordered part where value, package and rating
match; the rest keep the schematic's part or take a Yageo RC/CC part.

Co-Authored-By: Claude Opus 5.5 <noreply@anthropic.com>
Parts:
- D10, D9: MANUFACTURER Diodes -> Diodes Incorporated; MANUFACTURER_PN DT1240V3-04LP -> DT1240V3-04LP-7
- D4: MANUFACTURER Vishay -> Panjit International Inc.; MANUFACTURER_PN BAT54A -> BAT54A_R1_00001
- Q10, Q11, Q8, Q9: MANUFACTURER Diodes Inc -> Diodes Incorporated; MANUFACTURER_PN DMT4011LFG -> DMT4011LFG-13
- R22: MANUFACTURER ? -> YAGEO; MANUFACTURER_PN ? -> RC0402FR-071KL
- R24, R25, R26, R27: MANUFACTURER (none) -> YAGEO; MANUFACTURER_PN (none) -> RC0402JR-070RL
- U1: MANUFACTURER Analog Devices -> Analog Devices Inc.; MANUFACTURER_PN LTC1960CUHF -> LTC1960CUHF#PBF
Changed lines of the file:
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@@
 			)
 		)
-		(property "MANUFACTURER" "Diodes Inc"
+		(property "MANUFACTURER" "Diodes Incorporated"
 			(at 116.332 53.34 0)
 			(hide yes)
@@
 			)
 		)
-		(property "MANUFACTURER_PN" "DMT4011LFG"
+		(property "MANUFACTURER_PN" "DMT4011LFG-13"
 			(at 116.332 53.34 0)
 			(hide yes)
@@
 			)
 		)
-		(property "MANUFACTURER" "Diodes"
+		(property "MANUFACTURER" "Diodes Incorporated"
 			(at 314.452 194.31 0)
 			(hide yes)
@@
 			)
 		)
-		(property "MANUFACTURER_PN" "DT1240V3-04LP"
+		(property "MANUFACTURER_PN" "DT1240V3-04LP-7"
 			(at 314.452 194.31 0)
 			(hide yes)
@@
 			)
 		)
-		(property "MANUFACTURER" ""
+		(property "MANUFACTURER" "YAGEO"
 			(at 261.112 81.28 90)
 			(hide yes)
@@
 			)
 		)
-		(property "MANUFACTURER_PN" ""
+		(property "MANUFACTURER_PN" "RC0402JR-070RL"
 			(at 261.112 81.28 90)
 			(hide yes)
@@
 			)
 		)
-		(property "MANUFACTURER" "Diodes"
+		(property "MANUFACTURER" "Diodes Incorporated"
 			(at 314.452 99.06 0)
 			(hide yes)
@@
 			)
 		)
-		(property "MANUFACTURER_PN" "DT1240V3-04LP"
+		(property "MANUFACTURER_PN" "DT1240V3-04LP-7"
 			(at 314.452 99.06 0)
 			(hide yes)
@@
 			)
 		)
-		(property "MANUFACTURER" ""
+		(property "MANUFACTURER" "YAGEO"
 			(at 261.112 85.09 90)
 			(hide yes)
@@
 			)
 		)
-		(property "MANUFACTURER_PN" ""
+		(property "MANUFACTURER_PN" "RC0402JR-070RL"
 			(at 261.112 85.09 90)
 			(hide yes)
@@
 			)
 		)
-		(property "MANUFACTURER" ""
+		(property "MANUFACTURER" "YAGEO"
 			(at 261.112 172.72 90)
 			(hide yes)
@@
 			)
 		)
-		(property "MANUFACTURER_PN" ""
+		(property "MANUFACTURER_PN" "RC0402JR-070RL"
 			(at 261.112 172.72 90)
 			(hide yes)
@@
 			)
 		)
-		(property "MANUFACTURER" "Diodes Inc"
+		(property "MANUFACTURER" "Diodes Incorporated"
 			(at 96.012 53.34 0)
 			(hide yes)
@@
 			)
 		)
-		(property "MANUFACTURER_PN" "DMT4011LFG"
+		(property "MANUFACTURER_PN" "DMT4011LFG-13"
 			(at 96.012 53.34 0)
 			(hide yes)
@@
 			)
 		)
-		(property "MANUFACTURER" "Diodes Inc"
+		(property "MANUFACTURER" "Diodes Incorporated"
 			(at 115.062 144.78 0)
 			(hide yes)
@@
 			)
 		)
-		(property "MANUFACTURER_PN" "DMT4011LFG"
+		(property "MANUFACTURER_PN" "DMT4011LFG-13"
 			(at 115.062 144.78 0)
 			(hide yes)
@@
 			)
 		)
-		(property "MANUFACTURER" "?"
+		(property "MANUFACTURER" "YAGEO"
 			(at 51.054 108.712 0)
 			(hide yes)
@@
 			)
 		)
-		(property "MANUFACTURER_PN" "?"
+		(property "MANUFACTURER_PN" "RC0402FR-071KL"
 			(at 51.054 108.712 0)
 			(hide yes)
@@
 			)
 		)
-		(property "MANUFACTURER" "Analog Devices"
+		(property "MANUFACTURER" "Analog Devices Inc."
 			(at 154.432 113.03 0)
 			(hide yes)
@@
 			)
 		)
-		(property "MANUFACTURER_PN" "LTC1960CUHF"
+		(property "MANUFACTURER_PN" "LTC1960CUHF#PBF"
 			(at 154.432 113.03 0)
 			(hide yes)
@@
 			)
 		)
-		(property "MANUFACTURER" "Analog Devices"
+		(property "MANUFACTURER" "Analog Devices Inc."
 			(at 153.162 204.47 0)
 			(hide yes)
@@
 			)
 		)
-		(property "MANUFACTURER_PN" "LTC1960CUHF"
+		(property "MANUFACTURER_PN" "LTC1960CUHF#PBF"
 			(at 153.162 204.47 0)
 			(hide yes)
@@
 			)
 		)
-		(property "MANUFACTURER" "Vishay"
+		(property "MANUFACTURER" "Panjit International Inc."
 			(at 45.212 120.142 90)
 			(hide yes)
@@
 			)
 		)
-		(property "MANUFACTURER_PN" "BAT54A"
+		(property "MANUFACTURER_PN" "BAT54A_R1_00001"
 			(at 45.212 120.142 90)
 			(hide yes)
@@
 			)
 		)
-		(property "MANUFACTURER" "Diodes Inc"
+		(property "MANUFACTURER" "Diodes Incorporated"
 			(at 94.742 144.78 0)
 			(hide yes)
@@
 			)
 		)
-		(property "MANUFACTURER_PN" "DMT4011LFG"
+		(property "MANUFACTURER_PN" "DMT4011LFG-13"
 			(at 94.742 144.78 0)
 			(hide yes)
@@
 			)
 		)
-		(property "MANUFACTURER" ""
+		(property "MANUFACTURER" "YAGEO"
 			(at 261.112 176.53 90)
 			(hide yes)
@@
 			)
 		)
-		(property "MANUFACTURER_PN" ""
+		(property "MANUFACTURER_PN" "RC0402JR-070RL"
 			(at 261.112 176.53 90)
 			(hide yes)
