File: S08 IO Expander.kicad_sch (KiCad schematic)
At the start: 13 parts, among them Q23 BSS138, U11 PCAL9714

Commit message: Fill manufacturer part numbers from the 0.5.0 build orders
Set MANUFACTURER and MANUFACTURER_PN on every fitted part, in the
schematic and on the board. Unchanged parts take the exact part numbers
ordered for the 0.5.0 backup build (DigiKey list and Mouser basket);
changed parts reuse an ordered part where value, package and rating
match; the rest keep the schematic's part or take a Yageo RC/CC part.

Co-Authored-By: Claude Opus 5.5 <noreply@anthropic.com>
Parts:
- C58, C59: MANUFACTURER Yageo -> YAGEO
- R100, R99: MANUFACTURER ? -> YAGEO; MANUFACTURER_PN ? -> RC0402FR-07100KL
- R101: MANUFACTURER ? -> YAGEO; MANUFACTURER_PN ? -> RC0402FR-071M07L
- R93, R94: MANUFACTURER ? -> YAGEO; MANUFACTURER_PN ? -> RC0402FR-0710KL
- R95, R96, R97, R98: MANUFACTURER ? -> YAGEO; MANUFACTURER_PN ? -> RC0402JR-070RL
- U11: MANUFACTURER NXP -> NXP USA Inc.
Changed lines of the file:
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@@
 			)
 		)
-		(property "MANUFACTURER" "?"
+		(property "MANUFACTURER" "YAGEO"
 			(at 120.904 104.902 0)
 			(hide yes)
@@
 			)
 		)
-		(property "MANUFACTURER_PN" "?"
+		(property "MANUFACTURER_PN" "RC0402FR-071M07L"
 			(at 120.904 104.902 0)
 			(hide yes)
@@
 			)
 		)
-		(property "MANUFACTURER" "?"
+		(property "MANUFACTURER" "YAGEO"
 			(at 83.312 120.65 90)
 			(hide yes)
@@
 			)
 		)
-		(property "MANUFACTURER_PN" "?"
+		(property "MANUFACTURER_PN" "RC0402JR-070RL"
 			(at 83.312 120.65 90)
 			(hide yes)
@@
 			)
 		)
-		(property "MANUFACTURER" "?"
+		(property "MANUFACTURER" "YAGEO"
 			(at 120.904 93.472 0)
 			(hide yes)
@@
 			)
 		)
-		(property "MANUFACTURER_PN" "?"
+		(property "MANUFACTURER_PN" "RC0402FR-07100KL"
 			(at 120.904 93.472 0)
 			(hide yes)
@@
 			)
 		)
-		(property "MANUFACTURER" "?"
+		(property "MANUFACTURER" "YAGEO"
 			(at 139.954 158.242 0)
 			(hide yes)
@@
 			)
 		)
-		(property "MANUFACTURER_PN" "?"
+		(property "MANUFACTURER_PN" "RC0402FR-0710KL"
 			(at 139.954 158.242 0)
 			(hide yes)
@@
 			)
 		)
-		(property "MANUFACTURER" "?"
+		(property "MANUFACTURER" "YAGEO"
 			(at 138.684 118.872 0)
 			(hide yes)
@@
 			)
 		)
-		(property "MANUFACTURER_PN" "?"
+		(property "MANUFACTURER_PN" "RC0402FR-07100KL"
 			(at 138.684 118.872 0)
 			(hide yes)
@@
 			)
 		)
-		(property "MANUFACTURER" "Yageo"
+		(property "MANUFACTURER" "YAGEO"
 			(at 194.31 158.242 0)
 			(hide yes)
@@
 			)
 		)
-		(property "MANUFACTURER" "Yageo"
+		(property "MANUFACTURER" "YAGEO"
 			(at 181.61 158.242 0)
 			(hide yes)
@@
 			)
 		)
-		(property "MANUFACTURER" "?"
+		(property "MANUFACTURER" "YAGEO"
 			(at 83.312 110.49 90)
 			(hide yes)
@@
 			)
 		)
-		(property "MANUFACTURER_PN" "?"
+		(property "MANUFACTURER_PN" "RC0402JR-070RL"
 			(at 83.312 110.49 90)
 			(hide yes)
@@
 			)
 		)
-		(property "MANUFACTURER" "?"
+		(property "MANUFACTURER" "YAGEO"
 			(at 157.734 158.242 0)
 			(hide yes)
@@
 			)
 		)
-		(property "MANUFACTURER_PN" "?"
+		(property "MANUFACTURER_PN" "RC0402FR-0710KL"
 			(at 157.734 158.242 0)
 			(hide yes)
@@
 			)
 		)
-		(property "MANUFACTURER" "NXP"
+		(property "MANUFACTURER" "NXP USA Inc."
 			(at 181.102 137.16 0)
 			(hide yes)
@@
 			)
 		)
-		(property "MANUFACTURER" "?"
+		(property "MANUFACTURER" "YAGEO"
 			(at 83.312 102.87 90)
 			(hide yes)
@@
 			)
 		)
-		(property "MANUFACTURER_PN" "?"
+		(property "MANUFACTURER_PN" "RC0402JR-070RL"
 			(at 83.312 102.87 90)
 			(hide yes)
@@
 			)
 		)
-		(property "MANUFACTURER" "?"
+		(property "MANUFACTURER" "YAGEO"
 			(at 83.312 128.27 90)
 			(hide yes)
@@
 			)
 		)
-		(property "MANUFACTURER_PN" "?"
+		(property "MANUFACTURER_PN" "RC0402JR-070RL"
 			(at 83.312 128.27 90)
 			(hide yes)
