File: S07 Load Switch and I-Sense.kicad_sch (KiCad schematic)
At the start: 66 parts, among them Q20 BSS138, Q21 BSS138, Q22 BSS138, Q24 BSS138, U10 TLV9002IDSG, U6 TPS22811, U7 TPS22811, U8 TLV9002IDSG, U9 TPS22811

Commit message: DAQ UVLO bypass option R115; solder mask clearance 0.005 mm
R115 (0R, DNP) links nENDAQ to U6 EN/UVLO. Fitting it with Q24, R108 and
R109 removed drives DAQ like SBC and EXT: active high, no UVLO, with
R110 || R49 as the pull-down. Placed on top next to Q24. README, S07 note
and FIRMWARE_NOTES describe the option.

Co-Authored-By: Claude Opus 5.5 <noreply@anthropic.com>
Parts:
- added R115: 0R, Resistor_SMD:R_0402_1005Metric, symbol Device:R
Connections:
- net nENDAQ: now also R115.2
- net at Q24.3 (D), R108.1, R49.2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: now also R115.1
Changed lines of the file:
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@@
 		)
 	)
-	(text "DAQ (U6) is deliberately different from SBC and EXT; keep it.\nU6 has an 11 V undervoltage lockout: R108/R49 turn it on at\n11.2 V (10.8-11.7 V) and off at 10.2 V (9.8-10.7 V). That\ndivider must hold EN/UVLO, so the enable goes through Q24:\nnENDAQ is active LOW. High or floating (POR, expander in reset\nor unpowered) turns Q24 on and holds U6 in shutdown; low hands\nEN/UVLO to the divider. R109/R110 bias the gate from +12V, not\n+3V3MCU, so DAQ stays off when the MCU board is unpowered."
+	(text "DAQ (U6) is deliberately different from SBC and EXT; keep it.\nU6 has an 11 V undervoltage lockout: R108/R49 turn it on at\n11.2 V (10.8-11.7 V) and off at 10.2 V (9.8-10.7 V). That\ndivider must hold EN/UVLO, so the enable goes through Q24:\nnENDAQ is active LOW. High or floating (POR, expander in reset\nor unpowered) turns Q24 on and holds U6 in shutdown; low hands\nEN/UVLO to the divider. R109/R110 bias the gate from +12V, not\n+3V3MCU, so DAQ stays off when the MCU board is unpowered.\n\nBypass (assembly option): fit R115 0R and remove Q24, R108 and\nR109. nENDAQ then drives EN/UVLO directly, as on SBC and EXT:\nactive HIGH, no undervoltage lockout. R110 || R49 (8.3K) hold\nU6 off while the expander is in reset or unpowered."
 		(exclude_from_sim no)
 		(at 15.24 228.6 0)
@@
 		)
 	)
+	(symbol
+		(lib_id "Device:R")
+		(at 27.94 184.15 0)
+		(unit 1)
+		(body_style 1)
+		(exclude_from_sim no)
+		(in_bom yes)
+		(on_board yes)
+		(in_pos_files yes)
+		(dnp yes)
+		(property "Reference" "R115"
+			(at 26.924 182.88 0)
+			(show_name no)
+			(do_not_autoplace no)
+			(effects
+				(font
+					(size 1.27 1.27)
+				)
+				(justify right bottom)
+			)
+		)
+		(property "Value" "0R"
+			(at 26.924 185.42 0)
+			(show_name no)
+			(do_not_autoplace no)
+			(effects
+				(font
+					(size 1.27 1.27)
+				)
+				(justify right bottom)
+			)
+		)
+		(property "Footprint" "Resistor_SMD:R_0402_1005Metric"
+			(at 27.94 184.15 90)
+			(hide yes)
+			(show_name no)
+			(do_not_autoplace no)
+			(effects
+				(font
+					(size 1.27 1.27)
+				)
+			)
+		)
+		(property "Datasheet" ""
+			(at 27.94 184.15 90)
+			(hide yes)
+			(show_name no)
+			(do_not_autoplace no)
+			(effects
+				(font
+					(size 1.27 1.27)
+				)
+			)
+		)
+		(property "Description" "Resistor 0R 0402"
+			(at 27.94 184.15 90)
+			(hide yes)
+			(show_name no)
+			(do_not_autoplace no)
+			(effects
+				(font
+					(size 1.27 1.27)
+				)
+			)
+		)
+		(property "NOTE" ""
+			(at 26.924 182.88 0)
+			(hide yes)
+			(show_name no)
+			(do_not_autoplace no)
+			(effects
+				(font
+					(size 1.27 1.27)
+				)
+				(justify right bottom)
+			)
+		)
+		(property "PL_SORT_GROUP" "2.3"
+			(at 26.924 182.88 0)
+			(hide yes)
+			(show_name no)
+			(do_not_autoplace no)
+			(effects
+				(font
+					(size 1.27 1.27)
+				)
+				(justify right bottom)
+			)
+		)
+		(property "MANUFACTURER" "?"
+			(at 26.924 182.88 0)
+			(hide yes)
+			(show_name no)
+			(do_not_autoplace no)
+			(effects
+				(font
+					(size 1.27 1.27)
+				)
+				(justify right bottom)
+			)
+		)
+		(property "MANUFACTURER_PN" "?"
+			(at 26.924 182.88 0)
+			(hide yes)
+			(show_name no)
+			(do_not_autoplace no)
+			(effects
+				(font
+					(size 1.27 1.27)
+				)
+				(justify right bottom)
+			)
+		)
+		(property "ALTIUM_VALUE" "0R"
+			(at 26.924 182.88 0)
+			(hide yes)
+			(show_name no)
+			(do_not_autoplace no)
+			(effects
+				(font
+					(size 1.27 1.27)
+				)
+				(justify right bottom)
+			)
+		)
+		(property "ALTIUM_FOOTPRINT" "0402"
+			(at 26.924 187.96 0)
+			(show_name no)
+			(do_not_autoplace no)
+			(effects
+				(font
+					(size 1.27 1.27)
+				)
+				(justify right bottom)
+			)
+		)
+		(pin "2"
+		)
+		(pin "1"
+		)
+		(instances
+			(project "EVO2513"
+				(path "/44203427-0a3b-455b-9bb9-c1b577d179b3/3983715d-0555-40e9-9f86-7ce2617793ce"
+					(reference "R115")
+					(unit 1)
+				)
+			)
+		)
+	)
+	(wire
+		(pts
+			(xy 27.94 187.96) (xy 27.94 193.04)
+		)
+		(stroke
+			(width 0)
+			(type default)
+		)
+	)
+	(wire
+		(pts
+			(xy 27.94 180.34) (xy 27.94 177.8)
+		)
+		(stroke
+			(width 0)
+			(type default)
+		)
+	)
+	(wire
+		(pts
+			(xy 27.94 177.8) (xy 43.18 177.8)
+		)
+		(stroke
+			(width 0)
+			(type default)
+		)
+	)
+	(wire
+		(pts
+			(xy 43.18 177.8) (xy 43.18 185.42)
+		)
+		(stroke
+			(width 0)
+			(type default)
+		)
+	)
+	(wire
+		(pts
+			(xy 43.18 185.42) (xy 45.72 185.42)
+		)
+		(stroke
+			(width 0)
+			(type default)
+		)
+	)
+	(junction
+		(at 27.94 193.04)
+		(diameter 0)
+		(color 0 0 0 0)
+	)
+	(junction
+		(at 45.72 185.42)
+		(diameter 0)
+		(color 0 0 0 0)
+	)
 )

Commit message: Raise divider impedances, dim the PG LEDs, use standard diode lands
TI asks for a pull-up of at least 350 kOhm on EN/UVLO above 5 V.
R108 100K -> 619K and R49 12K -> 75K, both values already on the
BOM: turn-on 11.10 V (10.63-11.91 V worst case), off 10.09 V. 1M/120K
was rejected because leakage across 1M puts worst-case turn-on at
12.24 V, above the rail.

Q24 gate bias R109 100K -> 1.07M and R110 27K -> 390K: +12V draw
94 -> 8.2 uA, gate 3.2 V at 12 V and under 4 V worst case at the
14.7 V OVLO limit. The R115 bypass pull-down is now 62.9K.

PGTH dividers R59/R61/R76 100K -> 390K and R60/R62/R77 13K -> 51K:
PG at 10.38 V (11.17 V worst case), 23.5 uA at threshold to meet TI's
20x PGTH leakage rule. 390K is the only new BOM value.

PG LED resistors R67/R68/R81 2.2K -> 4.7K, about 0.9 mA less on
battery with all rails up.

D1, D4, D6-D10 and LED1-LED4 move from imported Altium lands to KiCad
standard footprints (D_SMB, D_SMA, SOT-23, Diodes_UDFN-10, LED_0603),
in place with the same nets; the LEDs turn 180 deg for pad 1. Drops
the 8 thin LED A/C silk warnings. Five unused imported footprints
removed. Nearby parts and tracks adjusted for the new lands.

Keep the GND planes free of power copper, as on the original: remove
the SW1/L2 and SW2 strip zones and the small +12V (via block by R115)
and U5 ISNSP (under Q18's drain) zones from In1/In3/In5/In6. They
carried no current; GND gains about 0.8 mm2 on In1, 3.5 mm2 on In3
and In5 and 3.7 mm2 on In6 under the power stage.

Remove the 347 via-block octagons the Altium import left as copper
graphic polygons (gr_poly) on B.Cu and In1-In6, one 1.2 x 1.8 mm
octagon per six-via block per layer. As drawings they bypassed zone
rules, and on the GND layers they were net islands in the pour,
including the charger switch node. None carried current: same-net
pours connect the vias solid, and DRC finds 0 unconnected. GND gains
about 26 mm2 on In1, 21 mm2 on In3 and In5, 18 mm2 on In6 and 27 mm2
on B.Cu.

Rename TPS22811 pin 2 to nEN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
Parts:
- D6, D7, D8: footprint EVO2513-0_5_0-import-fps:Diode DO-214AC SMA -> Diode_SMD:D_SMA
- LED2, LED3, LED4: footprint EVO2513-0_5_0-import-fps:LED 0603 H0-7 (C) -> LED_SMD:LED_0603_1608Metric
- R108: value 100K -> 619K; ALTIUM_VALUE 100K -> 619K
- R109: value 100K -> 1.07M; ALTIUM_VALUE 100K -> 1.07M
- R110: value 27K -> 390K; ALTIUM_VALUE 27K -> 390K
- R49: value 12K -> 75K; ALTIUM_VALUE 12K -> 75K
- R59, R61, R76: value 100K -> 390K; ALTIUM_VALUE 100K -> 390K
- R60, R62, R77: value 13K -> 51K; ALTIUM_VALUE 13K -> 51K
- R67, R68, R81: value 2.2K -> 4.7K; ALTIUM_VALUE 2.2K -> 4.7K
Other:
- note added: "DAQ (U6) is deliberately different from SBC and EXT. U6 has an 11 V undervoltage lockout: R108/R49 turn it on at 11.1 V (10.6-11.9 V) and off at 10.1 V (9.7-10.9 V). That divider must hold EN/UVLO, so the enable goes through Q24: nENDAQ is active LOW. High or floating (POR, expander in reset or unpowered) turns Q24 on and holds U6 in shutdown; low hands EN/UVLO to the divider. R109/R110 bias the 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"
- note added: "Overvoltage lockout: R90/R91/R92 1.07M with R51/R52/R70 100K on nEN/OVLO. Off above 14.0 V (13.4-14.7 V), back on below 12.75 V (12.2-13.4 V), so a tripped switch always recovers on the 12.03 V rail. PGTH dividers R59/R61/R76 390K over R60/R62/R77 51K: PG at 10.38 V (11.17 V worst case); 23.5 uA at threshold, over TI's 20x PGTH leakage."
- note removed: "DAQ (U6) is deliberately different from SBC and EXT; keep it. U6 has an 11 V undervoltage lockout: R108/R49 turn it on at 11.2 V (10.8-11.7 V) and off at 10.2 V (9.8-10.7 V). That divider must hold EN/UVLO, so the enable goes through Q24: nENDAQ is active LOW. High or floating (POR, expander in reset or unpowered) turns Q24 on and holds U6 in shutdown; low hands EN/UVLO to the divider. R109/R110 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"
- note removed: "Overvoltage lockout: R90/R91/R92 1.07M with R51/R52/R70 100K on nEN/OVLO. Off above 14.0 V (13.4-14.7 V), back on below 12.75 V (12.2-13.4 V), so a tripped switch always recovers on the 12.03 V rail. PGTH dividers R59/R61/R76 100K over R60/R62/R77 13K: PG at 10.43 V (10.93 V worst case); the low impedance keeps the PGTH pin leakage small."
- moved on the sheet: R108

Commit message: Fill manufacturer part numbers from the 0.5.0 build orders
Set MANUFACTURER and MANUFACTURER_PN on every fitted part, in the
schematic and on the board. Unchanged parts take the exact part numbers
ordered for the 0.5.0 backup build (DigiKey list and Mouser basket);
changed parts reuse an ordered part where value, package and rating
match; the rest keep the schematic's part or take a Yageo RC/CC part.

Co-Authored-By: Claude Opus 5.5 <noreply@anthropic.com>
Parts:
- C44, C45, C48, C49, C50, C54: MANUFACTURER ? -> Samsung Electro-Mechanics; MANUFACTURER_PN ? -> CL10A105KB8NNNC
- C46, C47, C51, C52, C53, R54: MANUFACTURER Yageo -> YAGEO
- C56: MANUFACTURER ?? -> YAGEO; MANUFACTURER_PN ?? -> CC0603KRX5R6BB106
- D6, D7, D8: MANUFACTURER_PN B340A -> B340A-13-F
- LED2, LED3, LED4: MANUFACTURER Everlight -> Everlight Electronics Co Ltd; MANUFACTURER_PN QTLP600C-4 -> QTLP600C4TR
- R108: MANUFACTURER ? -> YAGEO; MANUFACTURER_PN ? -> RC0402FR-07619KL
- R109, R90, R91, R92: MANUFACTURER ? -> YAGEO; MANUFACTURER_PN ? -> RC0402FR-071M07L
- R110, R59, R61, R76: MANUFACTURER ? -> YAGEO; MANUFACTURER_PN ? -> RC0402FR-07390KL
- R115: MANUFACTURER ? -> YAGEO; MANUFACTURER_PN ? -> RC0402JR-070RL
- R49: MANUFACTURER ? -> YAGEO; MANUFACTURER_PN ? -> RC0402FR-0775KL
- R50, R51, R52, R63, R65, R69, R70, R78: MANUFACTURER ? -> YAGEO; MANUFACTURER_PN ? -> RC0402FR-07100KL
- R53, R71: MANUFACTURER ? -> YAGEO; MANUFACTURER_PN ? -> RC0402FR-071KL
- R55, R56, R72, R73, R75: MANUFACTURER ? -> YAGEO; MANUFACTURER_PN ? -> RC0402FR-0710KL
- R57, R58, R74: MANUFACTURER ? -> YAGEO; MANUFACTURER_PN ? -> RC0402FR-0721K5L
- R60, R62, R77: MANUFACTURER (none) -> YAGEO; MANUFACTURER_PN (none) -> RC0402FR-0751KL
- R64, R66, R79, R80: MANUFACTURER ? -> YAGEO; MANUFACTURER_PN ? -> RC0402FR-07100RL
- R67, R68, R81: MANUFACTURER ? -> YAGEO; MANUFACTURER_PN ? -> RC0402FR-074K7L
- U10, U8: MANUFACTURER_PN TLV9002IDSG -> TLV9002IDSGR

Commit message: Move capacitors to currently available part numbers
C32 to Murata GRM219R61C226ME15L (GRM21BR61C226ME44L is no longer
generally available), C39 to Yageo CC0805KPX7R9BB102, the 1 uF 0603
caps to Murata GRT188R61H105KE13D, and the 10 uF 1210 caps to Taiyo
Yuden UMK325AB7106KMHP.

Co-Authored-By: Claude Opus 5.5 <noreply@anthropic.com>
Parts:
- C44, C45, C48, C49, C50, C54: MANUFACTURER Samsung Electro-Mechanics -> Murata Electronics; MANUFACTURER_PN CL10A105KB8NNNC -> GRT188R61H105KE13D
Changed lines of the file:
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@@
 			)
 		)
-		(property "MANUFACTURER" "Samsung Electro-Mechanics"
+		(property "MANUFACTURER" "Murata Electronics"
 			(at 55.88 80.772 0)
 			(hide yes)
@@
 			)
 		)
-		(property "MANUFACTURER_PN" "CL10A105KB8NNNC"
+		(property "MANUFACTURER_PN" "GRT188R61H105KE13D"
 			(at 55.88 80.772 0)
 			(hide yes)
@@
 			)
 		)
-		(property "MANUFACTURER" "Samsung Electro-Mechanics"
+		(property "MANUFACTURER" "Murata Electronics"
 			(at 53.34 207.772 0)
 			(hide yes)
@@
 			)
 		)
-		(property "MANUFACTURER_PN" "CL10A105KB8NNNC"
+		(property "MANUFACTURER_PN" "GRT188R61H105KE13D"
 			(at 53.34 207.772 0)
 			(hide yes)
@@
 			)
 		)
-		(property "MANUFACTURER" "Samsung Electro-Mechanics"
+		(property "MANUFACTURER" "Murata Electronics"
 			(at 224.79 79.502 0)
 			(hide yes)
@@
 			)
 		)
-		(property "MANUFACTURER_PN" "CL10A105KB8NNNC"
+		(property "MANUFACTURER_PN" "GRT188R61H105KE13D"
 			(at 224.79 79.502 0)
 			(hide yes)
@@
 			)
 		)
-		(property "MANUFACTURER" "Samsung Electro-Mechanics"
+		(property "MANUFACTURER" "Murata Electronics"
 			(at 171.45 50.292 0)
 			(hide yes)
@@
 			)
 		)
-		(property "MANUFACTURER_PN" "CL10A105KB8NNNC"
+		(property "MANUFACTURER_PN" "GRT188R61H105KE13D"
 			(at 171.45 50.292 0)
 			(hide yes)
@@
 			)
 		)
-		(property "MANUFACTURER" "Samsung Electro-Mechanics"
+		(property "MANUFACTURER" "Murata Electronics"
 			(at 168.91 177.292 0)
 			(hide yes)
@@
 			)
 		)
-		(property "MANUFACTURER_PN" "CL10A105KB8NNNC"
+		(property "MANUFACTURER_PN" "GRT188R61H105KE13D"
 			(at 168.91 177.292 0)
 			(hide yes)
@@
 			)
 		)
-		(property "MANUFACTURER" "Samsung Electro-Mechanics"
+		(property "MANUFACTURER" "Murata Electronics"
 			(at 340.36 49.022 0)
 			(hide yes)
@@
 			)
 		)
-		(property "MANUFACTURER_PN" "CL10A105KB8NNNC"
+		(property "MANUFACTURER_PN" "GRT188R61H105KE13D"
 			(at 340.36 49.022 0)
 			(hide yes)
